File: Eagle/Wordclock/WordclockKopie.brd (EAGLE design)
At the start: 160 x 100 mm, 231 parts

Commit message: Wordclock Matrix gelayoutet
Matrix alle Zeilen einzeln gelautet, Zeilen sind noch nicht verbunden
Parts:
- removed C111, C112, C113, C114: 100n, rcl:C1310
- removed L111, L112, L113, L114: WS2812B, adafruit:WS2812B
Connections:
- removed net INROW1: L1.4-DIN
- removed net N$12: L112.4-DIN, L113.2-DOUT
- removed net N$25: L111.4-DIN, L112.2-DOUT
- removed net N$26: L111.2-DOUT, L114.4-DIN
- removed net OUTGES: L114.2-DOUT
- removed net OUTROW1: L11.2-DOUT, L12.4-DIN
- removed net OUTROW10: L110.2-DOUT, L113.4-DIN
- removed net OUTROW2: L22.2-DOUT, L23.4-DIN
- removed net OUTROW3: L33.2-DOUT, L34.4-DIN
- removed net OUTROW4: L44.2-DOUT, L45.4-DIN
- removed net OUTROW5: L55.2-DOUT, L56.4-DIN
- removed net OUTROW6: L66.2-DOUT, L67.4-DIN
- removed net OUTROW7: L77.2-DOUT, L78.4-DIN
- removed net OUTROW8: L88.2-DOUT, L89.4-DIN
- removed net OUTROW9: L100.4-DIN, L99.2-DOUT
- net +5V: no longer C111.1, C112.1, C113.1, C114.1, L111.1-VDD, L112.1-VDD, L113.1-VDD, L114.1-VDD
- net GND: no longer C111.2, C112.2, C113.2, C114.2, L111.3-GND, L112.3-GND, L113.3-GND, L114.3-GND
