File: Eagle/Wordclock/WordclockKopie.sch (EAGLE design)
At the start: 231 parts

Commit message: Wordclock Matrix gelayoutet
Matrix alle Zeilen einzeln gelautet, Zeilen sind noch nicht verbunden
Parts:
- removed C111, C112, C113, C114: 100n, rcl:C-EUC1310
- removed L111, L112, L113, L114: WS2812B, adafruit:WS2812B
Connections:
- removed net INROW1: L1.DIN
- removed net N$12: L112.DIN, L113.DOUT
- removed net N$25: L111.DIN, L112.DOUT
- removed net N$26: L111.DOUT, L114.DIN
- removed net OUTGES: L114.DOUT
- removed net OUTROW1: L11.DOUT, L12.DIN
- removed net OUTROW10: L110.DOUT, L113.DIN
- removed net OUTROW2: L22.DOUT, L23.DIN
- removed net OUTROW3: L33.DOUT, L34.DIN
- removed net OUTROW4: L44.DOUT, L45.DIN
- removed net OUTROW5: L55.DOUT, L56.DIN
- removed net OUTROW6: L66.DOUT, L67.DIN
- removed net OUTROW7: L77.DOUT, L78.DIN
- removed net OUTROW8: L88.DOUT, L89.DIN
- removed net OUTROW9: L100.DIN, L99.DOUT
- net +5V: no longer C111.1, C112.1, C113.1, C114.1, L111.VDD, L112.VDD, L113.VDD, L114.VDD
- net GND: no longer C111.2, C112.2, C113.2, C114.2, L111.GND, L112.GND, L113.GND, L114.GND
