File: Eagle/Wordclock/Wordclock.brd (EAGLE design)
At the start: 160 x 100 mm, 74 parts, among them IC1 74HC595D, IC2 74HC595D, IC3 74HC595D, IC4 74HC595D, IC5 74HC595D, IC6 74HC595D, IC7 74HC595D, IC8 74HC595D

Commit message: Eagle Adafruit added
Parts:
- added LED65, LED66, LED67, LED68: WS2812B, WS2812B:WS2812B
- added Q1: (no value), special:Q
Connections:
- new net N$82: Q1.1, S+1.1
- new net N$83: Q1.2, S+1.2
- new net N$85: LED65.DOUT, LED66.DIN
- new net N$86: LED66.DOUT, LED67.DIN
- new net N$87: LED67.DOUT, LED68.DIN
- new net VDD: LED65.VDD, LED66.VDD, LED67.VDD, LED68.VDD
- net GND: now also LED65.VSS, LED66.VSS, LED67.VSS, LED68.VSS
- net N$81: now also S+1.4
Changed lines of the file:
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@@
 <layer number="54" name="bGND_GNDA" color="1" fill="9" visible="no" active="no"/>
 <layer number="56" name="wert" color="7" fill="1" visible="yes" active="yes"/>
+<layer number="57" name="tCAD" color="7" fill="1" visible="no" active="no"/>
 <layer number="90" name="Modules" color="5" fill="1" visible="no" active="no"/>
 <layer number="91" name="Nets" color="2" fill="1" visible="no" active="no"/>
@@
 <layer number="109" name="fp9" color="7" fill="1" visible="yes" active="yes"/>
 <layer number="110" name="fp0" color="7" fill="1" visible="yes" active="yes"/>
+<layer number="111" name="LPC17xx" color="7" fill="1" visible="yes" active="yes"/>
+<layer number="112" name="tSilk" color="7" fill="1" visible="yes" active="yes"/>
 <layer number="116" name="Patch_BOT" color="9" fill="4" visible="yes" active="yes"/>
 <layer number="121" name="_tsilk" color="7" fill="1" visible="yes" active="yes"/>
@@
 <layer number="123" name="tTestmark" color="7" fill="1" visible="yes" active="yes"/>
 <layer number="124" name="bTestmark" color="7" fill="1" visible="yes" active="yes"/>
+<layer number="125" name="_tNames" color="7" fill="1" visible="yes" active="yes"/>
+<layer number="126" name="_bNames" color="7" fill="1" visible="yes" active="yes"/>
+<layer number="127" name="_tValues" color="7" fill="1" visible="yes" active="yes"/>
+<layer number="128" name="_bValues" color="7" fill="1" visible="yes" active="yes"/>
 <layer number="131" name="tAdjust" color="7" fill="1" visible="yes" active="yes"/>
 <layer number="132" name="bAdjust" color="7" fill="1" visible="yes" active="yes"/>
 <layer number="144" name="Drill_legend" color="7" fill="1" visible="yes" active="yes"/>
+<layer number="150" name="Notes" color="7" fill="1" visible="no" active="yes"/>
 <layer number="151" name="HeatSink" color="7" fill="1" visible="yes" active="yes"/>
+<layer number="152" name="_bDocu" color="7" fill="1" visible="yes" active="yes"/>
+<layer number="153" name="FabDoc1" color="6" fill="1" visible="no" active="no"/>
+<layer number="154" name="FabDoc2" color="2" fill="1" visible="no" active="no"/>
+<layer number="155" name="FabDoc3" color="7" fill="15" visible="no" active="no"/>
 <layer number="199" name="Contour" color="7" fill="1" visible="yes" active="yes"/>
 <layer number="200" name="200bmp" color="1" fill="10" visible="no" active="no"/>
@@
 <layer number="215" name="215bmp" color="7" fill="1" visible="yes" active="yes"/>
 <layer number="216" name="216bmp" color="7" fill="1" visible="yes" active="yes"/>
+<layer number="217" name="217bmp" color="18" fill="1" visible="no" active="no"/>
+<layer number="218" name="218bmp" color="19" fill="1" visible="no" active="no"/>
+<layer number="219" name="219bmp" color="20" fill="1" visible="no" active="no"/>
+<layer number="220" name="220bmp" color="21" fill="1" visible="no" active="no"/>
+<layer number="221" name="221bmp" color="22" fill="1" visible="no" active="no"/>
+<layer number="222" name="222bmp" color="23" fill="1" visible="no" active="no"/>
+<layer number="223" name="223bmp" color="24" fill="1" visible="no" active="no"/>
+<layer number="224" name="224bmp" color="25" fill="1" visible="no" active="no"/>
+<layer number="248" name="Housing" color="7" fill="1" visible="yes" active="yes"/>
+<layer number="249" name="Edge" color="7" fill="1" visible="yes" active="yes"/>
 <layer number="250" name="Descript" color="7" fill="1" visible="no" active="no"/>
 <layer number="251" name="SMDround" color="7" fill="1" visible="no" active="no"/>
@@
 <element name="S+1" library="eagle-library-edeca.net-v5" package="DIL8" value="DS1337+" x="-60.96" y="-24.13"/>
 <element name="U$1" library="eagle-library-edeca.net-v5" package="MINI-USB" value="MINI-USB" x="-87.63" y="-21.59"/>
+<element name="Q1" library="special" package="Q" value="" x="-44.45" y="-34.29"/>
+<element name="LED65" library="WS2812B" package="WS2812B" value="WS2812B" x="-81.28" y="-41.91"/>
+<element name="LED66" library="WS2812B" package="WS2812B" value="WS2812B" x="-109.22" y="-38.1"/>
+<element name="LED67" library="WS2812B" package="WS2812B" value="WS2812B" x="-118.11" y="-40.64"/>
+<element name="LED68" library="WS2812B" package="WS2812B" value="WS2812B" x="-128.27" y="-48.26"/>
 </elements>
 <signals>
@@
 <contactref element="IC7" pad="8"/>
 <contactref element="IC8" pad="8"/>
+<contactref element="LED65" pad="VSS"/>
+<contactref element="LED66" pad="VSS"/>
+<contactref element="LED67" pad="VSS"/>
+<contactref element="LED68" pad="VSS"/>
+<wire x1="-116.11" y1="-42.34" x2="-126.27" y2="-49.96" width="0" layer="19" extent="1-1"/>
+<wire x1="-107.22" y1="-39.8" x2="-116.11" y2="-42.34" width="0" layer="19" extent="1-1"/>
+<wire x1="-79.28" y1="-43.61" x2="-107.22" y2="-39.8" width="0" layer="19" extent="1-1"/>
+<wire x1="-56.515" y1="2.0066" x2="-79.28" y2="-43.61" width="0" layer="19" extent="1-1"/>
 <wire x1="-56.515" y1="10.8966" x2="-56.515" y2="2.0066" width="0" layer="19" extent="1-1"/>
 <wire x1="-42.545" y1="2.0066" x2="-56.515" y2="2.0066" width="0" layer="19" extent="1-1"/>
@@
 <wire x1="-28.575" y1="2.0066" x2="-42.545" y2="2.0066" width="0" layer="19" extent="1-1"/>
 <wire x1="-28.575" y1="10.8966" x2="-28.575" y2="2.0066" width="0" layer="19" extent="1-1"/>
-<wire x1="1.905" y1="-3.0734" x2="-28.575" y2="2.0066" width="0" layer="19" extent="1-1"/>
-<wire x1="-14.605" y1="10.8966" x2="1.905" y2="-3.0734" width="0" layer="19" extent="1-1"/>
+<wire x1="-14.605" y1="10.8966" x2="-28.575" y2="10.8966" width="0" layer="19" extent="1-1"/>
+<wire x1="1.905" y1="-3.0734" x2="-14.605" y2="10.8966" width="0" layer="19" extent="1-1"/>
 </signal>
 <signal name="VCC">
@@
 <signal name="N$81">
 <contactref element="U$1" pad="5"/>
+<contactref element="S+1" pad="4"/>
+<wire x1="-57.15" y1="-27.94" x2="-85.38" y2="-23.19" width="0" layer="19" extent="1-1"/>
+</signal>
+<signal name="N$82">
+<contactref element="Q1" pad="1"/>
+<contactref element="S+1" pad="1"/>
+<wire x1="-64.77" y1="-27.94" x2="-46.99" y2="-41.91" width="0" layer="19" extent="1-1"/>
+</signal>
+<signal name="N$83">
+<contactref element="Q1" pad="2"/>
+<contactref element="S+1" pad="2"/>
+<wire x1="-62.23" y1="-27.94" x2="-41.91" y2="-41.91" width="0" layer="19" extent="1-1"/>
+</signal>
+<signal name="VDD">
+<contactref element="LED65" pad="VDD"/>
+<contactref element="LED66" pad="VDD"/>
+<contactref element="LED67" pad="VDD"/>
+<contactref element="LED68" pad="VDD"/>
+<wire x1="-120.11" y1="-38.94" x2="-130.27" y2="-46.56" width="0" layer="19" extent="1-1"/>
+<wire x1="-111.22" y1="-36.4" x2="-120.11" y2="-38.94" width="0" layer="19" extent="1-1"/>
+<wire x1="-83.28" y1="-40.21" x2="-111.22" y2="-36.4" width="0" layer="19" extent="1-1"/>
+</signal>
+<signal name="N$85">
+<contactref element="LED65" pad="DOUT"/>
+<contactref element="LED66" pad="DIN"/>
+<wire x1="-83.28" y1="-43.61" x2="-107.22" y2="-36.4" width="0" layer="19" extent="1-1"/>
+</signal>
+<signal name="N$86">
+<contactref element="LED66" pad="DOUT"/>
+<contactref element="LED67" pad="DIN"/>
+<wire x1="-111.22" y1="-39.8" x2="-116.11" y2="-38.94" width="0" layer="19" extent="1-1"/>
+</signal>
+<signal name="N$87">
+<contactref element="LED67" pad="DOUT"/>
+<contactref element="LED68" pad="DIN"/>
+<wire x1="-120.11" y1="-42.34" x2="-126.27" y2="-46.56" width="0" layer="19" extent="1-1"/>
 </signal>
 </signals>

Commit message: Eagle Fehler verbessert
Parts:
- removed IC2, IC3, IC4, IC5, IC6, IC7, IC8: 74HC595D, 74xx-eu:SO16
- removed LED10, LED11, LED12, LED13, LED14, LED15, LED16, LED17, LED18, LED19, LED20, LED21, LED22, LED23, LED24, LED25, LED26, LED27, LED28, LED29, LED30, LED31, LED32, LED33, LED34, LED35, LED36, LED37, LED38, LED39, LED40, LED41, LED42, LED43, LED44, LED45, LED46, LED47, LED48, LED49, LED50, LED51, LED52, LED53, LED54, LED55, LED56, LED57, LED58, LED59, LED60, LED61, LED62, LED63, LED64, LED9: (no value), led:LED3MM
- removed LED65, LED66, LED67, LED68: WS2812B, WS2812B:WS2812B
- added R1, R2, R3, R4, R5, R6, R7, R8: (no value), resistor:MINI_MELF-0102W
- LED1, LED2, LED3, LED4, LED5, LED6, LED7, LED8: device led:LED3MM -> led:SMARTLED-TTW
- moved LED6 173.4 mm to (-96.5, -41.9)
- moved LED7 147.6 mm to (-101.6, -41.9)
- moved LED8 144.9 mm to (-106.7, -41.9)
- moved LED1 128.6 mm to (-71.1, -41.9)
- moved U$1 127.6 mm to (16.5, 52.1)
- moved LED2 126.7 mm to (-76.2, -41.9)
- moved LED3 124.9 mm to (-81.3, -41.9)
- moved LED4 123.3 mm to (-86.4, -41.9)
- moved LED5 122.0 mm to (-91.4, -41.9)
- moved IC1 14.2 mm to (-5.08, 14.0)
Connections:
- removed net N$20 (its old number): IC3.1, LED18.A
- removed net N$21 (its old number): IC3.2, LED19.A
- removed net N$22: IC3.4, LED21.A
- removed net N$23: IC3.3, LED20.A
- removed net N$24: IC3.5, LED22.A
- removed net N$25: IC3.6, LED23.A
- removed net N$26: IC3.7, LED24.A
- removed net N$27: LED17.K, LED18.K, LED19.K, LED20.K, LED21.K, LED22.K, LED23.K, LED24.K
- removed net N$28: IC4.15, LED25.A
- removed net N$29: IC4.1, LED26.A
- removed net N$30: IC4.2, LED27.A
- removed net N$31: IC4.4, LED29.A
- removed net N$32: IC4.3, LED28.A
- removed net N$33: IC4.5, LED30.A
- removed net N$34: IC4.6, LED31.A
- removed net N$35: IC4.7, LED32.A
- removed net N$36: LED25.K, LED26.K, LED27.K, LED28.K, LED29.K, LED30.K, LED31.K, LED32.K
- removed net N$37: IC5.15, LED33.A
- removed net N$38: IC5.1, LED34.A
- removed net N$39: IC5.2, LED35.A
- removed net N$40: IC5.4, LED37.A
- removed net N$41: IC5.3, LED36.A
- removed net N$42: IC5.5, LED38.A
- removed net N$43: IC5.6, LED39.A
- removed net N$44: IC5.7, LED40.A
- removed net N$45: LED33.K, LED34.K, LED35.K, LED36.K, LED37.K, LED38.K, LED39.K, LED40.K
- removed net N$46: IC6.15, LED41.A
- removed net N$47: IC6.1, LED42.A
- removed net N$48: IC6.2, LED43.A
- removed net N$49: IC6.4, LED45.A
- removed net N$50: IC6.3, LED44.A
- removed net N$51: IC6.5, LED46.A
- removed net N$52: IC6.6, LED47.A
- removed net N$53: IC6.7, LED48.A
- removed net N$54: LED41.K, LED42.K, LED43.K, LED44.K, LED45.K, LED46.K, LED47.K, LED48.K
- removed net N$55: IC7.15, LED49.A
- removed net N$56: IC7.1, LED50.A
- removed net N$57: IC7.2, LED51.A
- removed net N$58: IC7.4, LED53.A
- removed net N$59: IC7.3, LED52.A
- removed net N$60: IC7.5, LED54.A
- removed net N$61: IC7.6, LED55.A
- removed net N$62: IC7.7, LED56.A
- removed net N$63: LED49.K, LED50.K, LED51.K, LED52.K, LED53.K, LED54.K, LED55.K, LED56.K
- removed net N$64: IC8.15, LED57.A
- removed net N$65: IC8.1, LED58.A
- removed net N$66: IC8.2, LED59.A
- removed net N$67: IC8.4, LED61.A
- removed net N$68: IC8.3, LED60.A
- removed net N$69: IC8.5, LED62.A
- removed net N$70: IC8.6, LED63.A
- removed net N$71: IC8.7, LED64.A
- removed net N$72: LED57.K, LED58.K, LED59.K, LED60.K, LED61.K, LED62.K, LED63.K, LED64.K
- removed net N$73: IC5.9, IC6.14
- removed net N$74: IC6.9, IC7.14
- removed net N$75: IC7.9, IC8.14
- removed net N$76: IC1.14, IC8.9
- removed net N$77: IC1.9, IC2.14
- removed net N$78: IC2.9, IC3.14
- removed net N$79: IC3.9, IC4.14
- removed net N$80: U$1.1
- removed net N$81: S+1.4, U$1.5
- removed net N$85: LED65.DOUT, LED66.DIN
- removed net N$86: LED66.DOUT, LED67.DIN
- removed net N$87: LED67.DOUT, LED68.DIN
- removed net VDD: LED65.VDD, LED66.VDD, LED67.VDD, LED68.VDD
- net GND: now also S+1.4, U$1.5; no longer IC2.8, IC3.8, IC4.8, IC5.8, IC6.8, IC7.8, IC8.8, LED65.VSS, LED66.VSS, LED67.VSS, LED68.VSS
- net N$1: now also IC1.4, LED5.A@1; no longer IC1.15, LED1.A
- net N$10: now also LED8.C@1, R8.1; no longer IC2.15, LED9.A
- net N$11: now also LED1.C@1, R1.1; no longer IC2.1, LED10.A
- net N$12: now also LED2.C@1, R2.1; no longer IC2.2, LED11.A
- net N$13: now also LED3.C@1, R3.1; no longer IC2.4, LED13.A
- net N$14: now also LED5.C@1, R5.1; no longer IC2.3, LED12.A
- net N$15: now also LED6.C@1, R6.1; no longer IC2.5, LED14.A
- net N$16: now also LED7.C@1, R7.1; no longer IC2.6, LED15.A
- net N$17: now also R1.2, R2.2, R3.2, R4.2, R5.2, R6.2, R7.2, R8.2; no longer IC2.7, LED16.A
- net N$18: now also IC1.14; no longer LED10.K, LED11.K, LED12.K, LED13.K, LED14.K, LED15.K, LED16.K, LED9.K
- net N$19: now also IC1.9; no longer IC3.15, LED17.A
- net N$2: now also IC1.5, LED6.A@1; no longer IC1.1, LED2.A
- net N$3: now also IC1.6, LED7.A@1; no longer IC1.2, LED3.A
- net N$4: now also IC1.7, LED8.A@1; no longer IC1.4, LED5.A
- net N$5: now also LED4.A@1; no longer LED4.A
- net N$6: now also IC1.2, LED3.A@1; no longer IC1.5, LED6.A
- net N$7: now also IC1.1, LED2.A@1; no longer IC1.6, LED7.A
- net N$8: now also IC1.15, LED1.A@1; no longer IC1.7, LED8.A
- net N$9: now also LED4.C@1, R4.1; no longer LED1.K, LED2.K, LED3.K, LED4.K, LED5.K, LED6.K, LED7.K, LED8.K
- net VCC: now also S+1.8, U$1.1; no longer IC2.16, IC3.16, IC4.16, IC5.16, IC6.16, IC7.16, IC8.16

Commit message: Eagle Änderung
Parts:
- moved IC1 95.5 mm to (-100.3, 20.3)
Connections:
- removed net N$17: R1.2, R2.2, R3.2, R4.2, R5.2, R6.2, R7.2, R8.2
- net GND: now also R1.2, R2.2, R3.2, R4.2, R5.2, R6.2, R7.2, R8.2
Changed lines of the file:
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@@
 </autorouter>
 <elements>
-<element name="IC1" library="74xx-eu" package="SO16" value="74HC595D" x="-5.08" y="13.97"/>
+<element name="IC1" library="74xx-eu" package="SO16" value="74HC595D" x="-100.33" y="20.32"/>
 <element name="S+1" library="eagle-library-edeca.net-v5" package="DIL8" value="DS1337+" x="-60.96" y="-24.13"/>
 <element name="Q1" library="special" package="Q" value="" x="-44.45" y="-34.29"/>
@@
 <contactref element="IC1" pad="8"/>
 <contactref element="S+1" pad="4"/>
-<wire x1="-0.635" y1="10.8966" x2="-57.15" y2="-27.94" width="0" layer="19" extent="1-1"/>
-<wire x1="18.76" y1="50.47" x2="-0.635" y2="10.8966" width="0" layer="19" extent="1-1"/>
+<contactref element="R8" pad="2"/>
+<contactref element="R1" pad="2"/>
+<contactref element="R2" pad="2"/>
+<contactref element="R3" pad="2"/>
+<contactref element="R4" pad="2"/>
+<contactref element="R5" pad="2"/>
+<contactref element="R6" pad="2"/>
+<contactref element="R7" pad="2"/>
+<wire x1="-105.73" y1="-69.85" x2="-105.73" y2="-73.66" width="0" layer="19" extent="1-1"/>
+<wire x1="-105.73" y1="-66.04" x2="-105.73" y2="-69.85" width="0" layer="19" extent="1-1"/>
+<wire x1="-105.73" y1="-62.23" x2="-105.73" y2="-66.04" width="0" layer="19" extent="1-1"/>
+<wire x1="-105.73" y1="-58.42" x2="-105.73" y2="-62.23" width="0" layer="19" extent="1-1"/>
+<wire x1="-105.73" y1="-54.61" x2="-105.73" y2="-58.42" width="0" layer="19" extent="1-1"/>
+<wire x1="-105.73" y1="-50.8" x2="-105.73" y2="-54.61" width="0" layer="19" extent="1-1"/>
+<wire x1="-105.73" y1="-46.99" x2="-105.73" y2="-50.8" width="0" layer="19" extent="1-1"/>
+<wire x1="-57.15" y1="-27.94" x2="-105.73" y2="-46.99" width="0" layer="19" extent="1-1"/>
+<wire x1="-95.885" y1="17.2466" x2="-57.15" y2="-27.94" width="0" layer="19" extent="1-1"/>
+<wire x1="18.76" y1="50.47" x2="-57.15" y2="-27.94" width="0" layer="19" extent="1-1"/>
 </signal>
 <signal name="N$1">
 <contactref element="IC1" pad="4"/>
 <contactref element="LED5" pad="A@1"/>
-<wire x1="-5.715" y1="10.8966" x2="-91.44" y2="-42.41" width="0" layer="19" extent="1-1"/>
+<wire x1="-100.965" y1="17.2466" x2="-91.44" y2="-42.41" width="0" layer="19" extent="1-1"/>
 </signal>
 <signal name="N$2">
 <contactref element="IC1" pad="5"/>
 <contactref element="LED6" pad="A@1"/>
-<wire x1="-4.445" y1="10.8966" x2="-96.52" y2="-42.41" width="0" layer="19" extent="1-1"/>
+<wire x1="-99.695" y1="17.2466" x2="-96.52" y2="-42.41" width="0" layer="19" extent="1-1"/>
 </signal>
 <signal name="N$3">
 <contactref element="IC1" pad="6"/>
 <contactref element="LED7" pad="A@1"/>
-<wire x1="-3.175" y1="10.8966" x2="-101.6" y2="-42.41" width="0" layer="19" extent="1-1"/>
+<wire x1="-98.425" y1="17.2466" x2="-101.6" y2="-42.41" width="0" layer="19" extent="1-1"/>
 </signal>
 <signal name="N$4">
 <contactref element="IC1" pad="7"/>
 <contactref element="LED8" pad="A@1"/>
-<wire x1="-1.905" y1="10.8966" x2="-106.68" y2="-42.41" width="0" layer="19" extent="1-1"/>
+<wire x1="-97.155" y1="17.2466" x2="-106.68" y2="-42.41" width="0" layer="19" extent="1-1"/>
 </signal>
 <signal name="N$5">
 <contactref element="IC1" pad="3"/>
 <contactref element="LED4" pad="A@1"/>
-<wire x1="-6.985" y1="10.8966" x2="-86.36" y2="-42.41" width="0" layer="19" extent="1-1"/>
+<wire x1="-102.235" y1="17.2466" x2="-86.36" y2="-42.41" width="0" layer="19" extent="1-1"/>
 </signal>
 <signal name="N$6">
 <contactref element="LED3" pad="A@1"/>
 <contactref element="IC1" pad="2"/>
-<wire x1="-8.255" y1="10.8966" x2="-81.28" y2="-42.41" width="0" layer="19" extent="1-1"/>
+<wire x1="-103.505" y1="17.2466" x2="-81.28" y2="-42.41" width="0" layer="19" extent="1-1"/>
 </signal>
 <signal name="N$7">
 <contactref element="IC1" pad="1"/>
 <contactref element="LED2" pad="A@1"/>
-<wire x1="-9.525" y1="10.8966" x2="-76.2" y2="-42.41" width="0" layer="19" extent="1-1"/>
+<wire x1="-104.775" y1="17.2466" x2="-76.2" y2="-42.41" width="0" layer="19" extent="1-1"/>
 </signal>
 <signal name="N$8">
 <contactref element="LED1" pad="A@1"/>
 <contactref element="IC1" pad="15"/>
-<wire x1="-8.255" y1="17.0434" x2="-71.12" y2="-42.41" width="0" layer="19" extent="1-1"/>
+<wire x1="-103.505" y1="23.3934" x2="-71.12" y2="-42.41" width="0" layer="19" extent="1-1"/>
 </signal>
 <signal name="N$9">
@@
 <wire x1="-101.6" y1="-41.41" x2="-107.63" y2="-69.85" width="0" layer="19" extent="1-1"/>
 </signal>
-<signal name="N$17">
-<contactref element="R8" pad="2"/>
-<contactref element="R1" pad="2"/>
-<contactref element="R2" pad="2"/>
-<contactref element="R3" pad="2"/>
-<contactref element="R4" pad="2"/>
-<contactref element="R5" pad="2"/>
-<contactref element="R6" pad="2"/>
-<contactref element="R7" pad="2"/>
-<wire x1="-105.73" y1="-69.85" x2="-105.73" y2="-73.66" width="0" layer="19" extent="1-1"/>
-<wire x1="-105.73" y1="-66.04" x2="-105.73" y2="-69.85" width="0" layer="19" extent="1-1"/>
-<wire x1="-105.73" y1="-62.23" x2="-105.73" y2="-66.04" width="0" layer="19" extent="1-1"/>
-<wire x1="-105.73" y1="-58.42" x2="-105.73" y2="-62.23" width="0" layer="19" extent="1-1"/>
-<wire x1="-105.73" y1="-54.61" x2="-105.73" y2="-58.42" width="0" layer="19" extent="1-1"/>
-<wire x1="-105.73" y1="-50.8" x2="-105.73" y2="-54.61" width="0" layer="19" extent="1-1"/>
-<wire x1="-105.73" y1="-46.99" x2="-105.73" y2="-50.8" width="0" layer="19" extent="1-1"/>
-</signal>
 <signal name="N$18">
 <contactref element="IC1" pad="14"/>
@@
 <contactref element="U$1" pad="1"/>
 <contactref element="S+1" pad="8"/>
-<wire x1="-9.525" y1="17.0434" x2="-64.77" y2="-20.32" width="0" layer="19" extent="1-1"/>
-<wire x1="18.76" y1="53.67" x2="-9.525" y2="17.0434" width="0" layer="19" extent="1-1"/>
+<wire x1="-104.775" y1="23.3934" x2="-64.77" y2="-20.32" width="0" layer="19" extent="1-1"/>
+<wire x1="18.76" y1="53.67" x2="-104.775" y2="23.3934" width="0" layer="19" extent="1-1"/>
 </signal>
 <signal name="N$20">
