File: Eagle/Wordclock/Wordclock.brd (EAGLE design)
At the start: 160 x 100 mm, 20 parts, among them IC1 74HC595D

Commit message: Eagel WS2812 added
Parts:
- removed IC1: 74HC595D, 74xx-eu:SO16
- removed LED1, LED2, LED3, LED4, LED5, LED6, LED7, LED8: (no value), led:SMARTLED-TTW
- removed R1, R2, R3, R4, R5, R6, R7, R8: (no value), resistor:MINI_MELF-0102W
- added C1, C10, C100, C101, C102, C103, C104, C105, C106, C107, C108, C109, C11, C110, C12, C13, C14, C15, C16, C17, C18, C19, C2, C20, C21, C22, C23, C24, C25, C26, C27, C28, C29, C3, C30, C31, C32, C33, C34, C35, C36, C37, C38, C39, C4, C40, C41, C42, C43, C44, C45, C46, C47, C48, C49, C5, C50, C51, C52, C53, C54, C55, C56, C57, C58, C59, C6, C60, C61, C62, C63, C64, C65, C66, C67, C68, C69, C7, C70, C71, C72, C73, C74, C75, C76, C77, C78, C79, C8, C80, C81, C82, C83, C84, C85, C86, C87, C88, C89, C9, C90, C91, C92, C93, C94, C95, C96, C97, C98, C99: 100n, rcl:C1310
- added L1, L10, L100, L101, L102, L103, L104, L105, L106, L107, L108, L109, L11, L110, L12, L13, L14, L15, L16, L17, L18, L19, L2, L20, L21, L22, L23, L24, L25, L26, L27, L28, L29, L3, L30, L31, L32, L33, L34, L35, L36, L37, L38, L39, L4, L40, L41, L42, L43, L44, L45, L46, L47, L48, L49, L5, L50, L51, L52, L53, L54, L55, L56, L57, L58, L59, L6, L60, L61, L62, L63, L64, L65, L66, L67, L68, L69, L7, L70, L71, L72, L73, L74, L75, L76, L77, L78, L79, L8, L80, L81, L82, L83, L84, L85, L86, L87, L88, L89, L9, L90, L91, L92, L93, L94, L95, L96, L97, L98, L99: WS2812B, adafruit:WS2812B
Connections:
- removed net N$11: LED1.C@1, R1.1
- new net +5V: C1.1, C10.1, C100.1, C101.1, C102.1, C103.1, C104.1, C105.1, C106.1, C107.1, C108.1, C109.1, C11.1, C110.1, C12.1, C13.1, C14.1, C15.1, C16.1, C17.1, C18.1, C19.1, C2.1, C20.1, C21.1, C22.1, C23.1, C24.1, C25.1, C26.1, C27.1, C28.1, C29.1, C3.1, C30.1, C31.1, C32.1, C33.1, C34.1, C35.1, C36.1, C37.1, C38.1, C39.1, C4.1, C40.1, C41.1, C42.1, C43.1, C44.1, C45.1, C46.1, C47.1, C48.1, C49.1, C5.1, C50.1, C51.1, C52.1, C53.1, C54.1, C55.1, C56.1, C57.1, C58.1, C59.1, C6.1, C60.1, C61.1, C62.1, C63.1, C64.1, C65.1, C66.1, C67.1, C68.1, C69.1, C7.1, C70.1, C71.1, C72.1, C73.1, C74.1, C75.1, C76.1, C77.1, C78.1, C79.1, C8.1, C80.1, C81.1, C82.1, C83.1, C84.1, C85.1, C86.1, C87.1, C88.1, C89.1, C9.1, C90.1, C91.1, C92.1, C93.1, C94.1, C95.1, C96.1, C97.1, C98.1, C99.1, L1.1-VDD, L10.1-VDD, L100.1-VDD, L101.1-VDD, L102.1-VDD, L103.1-VDD, L104.1-VDD, L105.1-VDD, L106.1-VDD, L107.1-VDD, L108.1-VDD, L109.1-VDD, L11.1-VDD, L110.1-VDD, L12.1-VDD, L13.1-VDD, L14.1-VDD, L15.1-VDD, L16.1-VDD, L17.1-VDD, L18.1-VDD, L19.1-VDD, L2.1-VDD, L20.1-VDD, L21.1-VDD, L22.1-VDD, L23.1-VDD, L24.1-VDD, L25.1-VDD, L26.1-VDD, L27.1-VDD, L28.1-VDD, L29.1-VDD, L3.1-VDD, L30.1-VDD, L31.1-VDD, L32.1-VDD, L33.1-VDD, L34.1-VDD, L35.1-VDD, L36.1-VDD, L37.1-VDD, L38.1-VDD, L39.1-VDD, L4.1-VDD, L40.1-VDD, L41.1-VDD, L42.1-VDD, L43.1-VDD, L44.1-VDD, L45.1-VDD, L46.1-VDD, L47.1-VDD, L48.1-VDD, L49.1-VDD, L5.1-VDD, L50.1-VDD, L51.1-VDD, L52.1-VDD, L53.1-VDD, L54.1-VDD, L55.1-VDD, L56.1-VDD, L57.1-VDD, L58.1-VDD, L59.1-VDD, L6.1-VDD, L60.1-VDD, L61.1-VDD, L62.1-VDD, L63.1-VDD, L64.1-VDD, L65.1-VDD, L66.1-VDD, L67.1-VDD, L68.1-VDD, L69.1-VDD, L7.1-VDD, L70.1-VDD, L71.1-VDD, L72.1-VDD, L73.1-VDD, L74.1-VDD, L75.1-VDD, L76.1-VDD, L77.1-VDD, L78.1-VDD, L79.1-VDD, L8.1-VDD, L80.1-VDD, L81.1-VDD, L82.1-VDD, L83.1-VDD, L84.1-VDD, L85.1-VDD, L86.1-VDD, L87.1-VDD, L88.1-VDD, L89.1-VDD, L9.1-VDD, L90.1-VDD, L91.1-VDD, L92.1-VDD, L93.1-VDD, L94.1-VDD, L95.1-VDD, L96.1-VDD, L97.1-VDD, L98.1-VDD, L99.1-VDD
- new net N$100: L90.2-DOUT, L91.4-DIN
- new net N$101: L91.2-DOUT, L92.4-DIN
- new net N$102: L92.2-DOUT, L93.4-DIN
- new net N$103: L93.2-DOUT, L94.4-DIN
- new net N$104: L94.2-DOUT, L95.4-DIN
- new net N$105: L95.2-DOUT, L96.4-DIN
- new net N$106: L96.2-DOUT, L97.4-DIN
- new net N$107: L97.2-DOUT, L98.4-DIN
- new net N$108: L98.2-DOUT, L99.4-DIN
- new net N$111: L100.2-DOUT, L101.4-DIN
- new net N$112: L101.2-DOUT, L102.4-DIN
- new net N$113: L102.2-DOUT, L103.4-DIN
- new net N$114: L103.2-DOUT, L104.4-DIN
- new net N$115: L104.2-DOUT, L105.4-DIN
- new net N$116: L105.2-DOUT, L106.4-DIN
- new net N$117: L106.2-DOUT, L107.4-DIN
- new net N$118: L107.2-DOUT, L108.4-DIN
- new net N$119: L108.2-DOUT, L109.4-DIN
- new net N$120: L109.2-DOUT, L110.4-DIN
- new net N$17: L16.2-DOUT, L17.4-DIN
- new net N$22: L19.2-DOUT, L20.4-DIN
- new net N$23: L20.2-DOUT, L21.4-DIN
- new net N$24: L21.2-DOUT, L22.4-DIN
- new net N$27: L23.2-DOUT, L24.4-DIN
- new net N$28: L24.2-DOUT, L25.4-DIN
- new net N$29: L25.2-DOUT, L26.4-DIN
- new net N$30: L26.2-DOUT, L27.4-DIN
- new net N$31: L27.2-DOUT, L28.4-DIN
- new net N$32: L28.2-DOUT, L29.4-DIN
- new net N$33: L29.2-DOUT, L30.4-DIN
- new net N$34: L30.2-DOUT, L31.4-DIN
- new net N$35: L31.2-DOUT, L32.4-DIN
- new net N$36: L32.2-DOUT, L33.4-DIN
- new net N$39: L34.2-DOUT, L35.4-DIN
- new net N$40: L35.2-DOUT, L36.4-DIN
- new net N$41: L36.2-DOUT, L37.4-DIN
- new net N$42: L37.2-DOUT, L38.4-DIN
- new net N$43: L38.2-DOUT, L39.4-DIN
- new net N$44: L39.2-DOUT, L40.4-DIN
- new net N$45: L40.2-DOUT, L41.4-DIN
- new net N$46: L41.2-DOUT, L42.4-DIN
- new net N$47: L42.2-DOUT, L43.4-DIN
- new net N$48: L43.2-DOUT, L44.4-DIN
- new net N$51: L45.2-DOUT, L46.4-DIN
- new net N$52: L46.2-DOUT, L47.4-DIN
- new net N$53: L47.2-DOUT, L48.4-DIN
- new net N$54: L48.2-DOUT, L49.4-DIN
- new net N$55: L49.2-DOUT, L50.4-DIN
- new net N$56: L50.2-DOUT, L51.4-DIN
- new net N$57: L51.2-DOUT, L52.4-DIN
- new net N$58: L52.2-DOUT, L53.4-DIN
- new net N$59: L53.2-DOUT, L54.4-DIN
- new net N$60: L54.2-DOUT, L55.4-DIN
- new net N$63: L56.2-DOUT, L57.4-DIN
- new net N$64: L57.2-DOUT, L58.4-DIN
- new net N$65: L58.2-DOUT, L59.4-DIN
- new net N$66: L59.2-DOUT, L60.4-DIN
- new net N$67: L60.2-DOUT, L61.4-DIN
- new net N$68: L61.2-DOUT, L62.4-DIN
- new net N$69: L62.2-DOUT, L63.4-DIN
- new net N$70: L63.2-DOUT, L64.4-DIN
- new net N$71: L64.2-DOUT, L65.4-DIN
- new net N$72: L65.2-DOUT, L66.4-DIN
- new net N$75: L67.2-DOUT, L68.4-DIN
- new net N$76: L68.2-DOUT, L69.4-DIN
- new net N$77: L69.2-DOUT, L70.4-DIN
- new net N$78: L70.2-DOUT, L71.4-DIN
- new net N$79: L71.2-DOUT, L72.4-DIN
- new net N$80: L72.2-DOUT, L73.4-DIN
- new net N$81: L73.2-DOUT, L74.4-DIN
- new net N$82: L74.2-DOUT, L75.4-DIN
- new net N$83: L75.2-DOUT, L76.4-DIN
- new net N$84: L76.2-DOUT, L77.4-DIN
- new net N$87: L78.2-DOUT, L79.4-DIN
- new net N$88: L79.2-DOUT, L80.4-DIN
- new net N$89: L80.2-DOUT, L81.4-DIN
- new net N$90: L81.2-DOUT, L82.4-DIN
- new net N$91: L82.2-DOUT, L83.4-DIN
- new net N$92: L83.2-DOUT, L84.4-DIN
- new net N$93: L84.2-DOUT, L85.4-DIN
- new net N$94: L85.2-DOUT, L86.4-DIN
- new net N$95: L86.2-DOUT, L87.4-DIN
- new net N$96: L87.2-DOUT, L88.4-DIN
- new net N$99: L89.2-DOUT, L90.4-DIN
- new net OUTROW1: L11.2-DOUT, L12.4-DIN
- new net OUTROW10: L110.2-DOUT
- new net OUTROW2: L22.2-DOUT, L23.4-DIN
- new net OUTROW3: L33.2-DOUT, L34.4-DIN
- new net OUTROW4: L44.2-DOUT, L45.4-DIN
- new net OUTROW5: L55.2-DOUT, L56.4-DIN
- new net OUTROW6: L66.2-DOUT, L67.4-DIN
- new net OUTROW7: L77.2-DOUT, L78.4-DIN
- new net OUTROW8: L88.2-DOUT, L89.4-DIN
- new net OUTROW9: L100.4-DIN, L99.2-DOUT
- net GND: now also C1.2, C10.2, C100.2, C101.2, C102.2, C103.2, C104.2, C105.2, C106.2, C107.2, C108.2, C109.2, C11.2, C110.2, C12.2, C13.2, C14.2, C15.2, C16.2, C17.2, C18.2, C19.2, C2.2, C20.2, C21.2, C22.2, C23.2, C24.2, C25.2, C26.2, C27.2, C28.2, C29.2, C3.2, C30.2, C31.2, C32.2, C33.2, C34.2, C35.2, C36.2, C37.2, C38.2, C39.2, C4.2, C40.2, C41.2, C42.2, C43.2, C44.2, C45.2, C46.2, C47.2, C48.2, C49.2, C5.2, C50.2, C51.2, C52.2, C53.2, C54.2, C55.2, C56.2, C57.2, C58.2, C59.2, C6.2, C60.2, C61.2, C62.2, C63.2, C64.2, C65.2, C66.2, C67.2, C68.2, C69.2, C7.2, C70.2, C71.2, C72.2, C73.2, C74.2, C75.2, C76.2, C77.2, C78.2, C79.2, C8.2, C80.2, C81.2, C82.2, C83.2, C84.2, C85.2, C86.2, C87.2, C88.2, C89.2, C9.2, C90.2, C91.2, C92.2, C93.2, C94.2, C95.2, C96.2, C97.2, C98.2, C99.2, L1.3-GND, L10.3-GND, L100.3-GND, L101.3-GND, L102.3-GND, L103.3-GND, L104.3-GND, L105.3-GND, L106.3-GND, L107.3-GND, L108.3-GND, L109.3-GND, L11.3-GND, L110.3-GND, L12.3-GND, L13.3-GND, L14.3-GND, L15.3-GND, L16.3-GND, L17.3-GND, L18.3-GND, L19.3-GND, L2.3-GND, L20.3-GND, L21.3-GND, L22.3-GND, L23.3-GND, L24.3-GND, L25.3-GND, L26.3-GND, L27.3-GND, L28.3-GND, L29.3-GND, L3.3-GND, L30.3-GND, L31.3-GND, L32.3-GND, L33.3-GND, L34.3-GND, L35.3-GND, L36.3-GND, L37.3-GND, L38.3-GND, L39.3-GND, L4.3-GND, L40.3-GND, L41.3-GND, L42.3-GND, L43.3-GND, L44.3-GND, L45.3-GND, L46.3-GND, L47.3-GND, L48.3-GND, L49.3-GND, L5.3-GND, L50.3-GND, L51.3-GND, L52.3-GND, L53.3-GND, L54.3-GND, L55.3-GND, L56.3-GND, L57.3-GND, L58.3-GND, L59.3-GND, L6.3-GND, L60.3-GND, L61.3-GND, L62.3-GND, L63.3-GND, L64.3-GND, L65.3-GND, L66.3-GND, L67.3-GND, L68.3-GND, L69.3-GND, L7.3-GND, L70.3-GND, L71.3-GND, L72.3-GND, L73.3-GND, L74.3-GND, L75.3-GND, L76.3-GND, L77.3-GND, L78.3-GND, L79.3-GND, L8.3-GND, L80.3-GND, L81.3-GND, L82.3-GND, L83.3-GND, L84.3-GND, L85.3-GND, L86.3-GND, L87.3-GND, L88.3-GND, L89.3-GND, L9.3-GND, L90.3-GND, L91.3-GND, L92.3-GND, L93.3-GND, L94.3-GND, L95.3-GND, L96.3-GND, L97.3-GND, L98.3-GND, L99.3-GND; no longer IC1.8, R1.2, R2.2, R3.2, R4.2, R5.2, R6.2, R7.2, R8.2
- net N$1: now also L1.2-DOUT, L2.4-DIN; no longer IC1.4, LED5.A@1
- net N$10: now also L10.2-DOUT, L11.4-DIN; no longer LED8.C@1, R8.1
- net N$12: now also L1.4-DIN; no longer LED2.C@1, R2.1
- net N$13: now also L12.2-DOUT, L13.4-DIN; no longer LED3.C@1, R3.1
- net N$14: now also L13.2-DOUT, L14.4-DIN; no longer LED5.C@1, R5.1
- net N$15: now also L14.2-DOUT, L15.4-DIN; no longer LED6.C@1, R6.1
- net N$16: now also L15.2-DOUT, L16.4-DIN; no longer LED7.C@1, R7.1
- net N$18: now also L17.2-DOUT, L18.4-DIN; no longer IC1.14
- net N$19: now also L18.2-DOUT, L19.4-DIN; no longer IC1.9
- net N$2: now also L2.2-DOUT, L3.4-DIN; no longer IC1.5, LED6.A@1
- net N$3: now also L3.2-DOUT, L4.4-DIN; no longer IC1.6, LED7.A@1
- net N$4: now also L4.2-DOUT, L5.4-DIN; no longer IC1.7, LED8.A@1
- net N$5: now also L6.2-DOUT, L7.4-DIN; no longer IC1.3, LED4.A@1
- net N$6: now also L5.2-DOUT, L6.4-DIN; no longer IC1.2, LED3.A@1
- net N$7: now also L7.2-DOUT, L8.4-DIN; no longer IC1.1, LED2.A@1
- net N$8: now also L8.2-DOUT, L9.4-DIN; no longer IC1.15, LED1.A@1
- net N$9: now also L10.4-DIN, L9.2-DOUT; no longer LED4.C@1, R4.1
- net VCC: no longer IC1.16, S+1.8
Routing:
- net GND: track 0.00 -> 75.7 mm
- net N$2: track 0.00 -> 6.63 mm
- net N$1: track 0.00 -> 6.63 mm
- net N$4: track 0.00 -> 6.63 mm
- net N$3: track 0.00 -> 6.63 mm

Commit message: WS2812 Layout versucht
Parts:
- added C111, C112, C113, C114: 100n, rcl:C1310
- added L111, L112, L113, L114: WS2812B, adafruit:WS2812B
- moved L6 81.0 mm to (23.9, -36.8)
- moved C1 10.8 mm to (-26.5, -42.1)
- moved C2 10.8 mm to (-16.3, -42.1)
- moved C3 10.8 mm to (-6.16, -42.1)
- moved C4 10.8 mm to (4.00, -42.1)
- moved C5 10.8 mm to (14.2, -42.1)
- moved L1 10.8 mm to (-26.5, -38.3)
- moved L2 10.8 mm to (-16.3, -38.3)
- moved L3 10.8 mm to (-6.16, -38.3)
- moved L4 10.8 mm to (4.00, -38.3)
- moved L5 10.8 mm to (14.2, -38.3)
- moved L20 8.75 mm to (-38.2, -121.9)
Connections:
- net N$12 renamed INROW1
- new net N$12: L112.4-DIN, L113.2-DOUT
- new net N$25: L111.4-DIN, L112.2-DOUT
- new net N$26: L111.2-DOUT, L114.4-DIN
- new net OUTGES: L114.2-DOUT
- net +5V: now also C111.1, C112.1, C113.1, C114.1, L111.1-VDD, L112.1-VDD, L113.1-VDD, L114.1-VDD
- net GND: now also C111.2, C112.2, C113.2, C114.2, L111.3-GND, L112.3-GND, L113.3-GND, L114.3-GND
- net OUTROW10: now also L113.4-DIN
Routing:
- net GND: track 75.7 -> 69.5 mm

Commit message: Wordclock Matrix gelayoutet
Matrix alle Zeilen einzeln gelautet, Zeilen sind noch nicht verbunden
Parts:
- removed C111, C112, C113, C114: 100n, rcl:C1310
- removed L111, L112, L113, L114: WS2812B, adafruit:WS2812B
- moved L98 260.8 mm to (77.9, -68.6), turned to 270 degrees
- moved L99 260.7 mm to (86.5, -68.6), turned to 270 degrees
- moved C99 259.9 mm to (90.8, -67.1), turned to 90 degrees
- moved L108 259.7 mm to (69.2, -77.2), turned to 270 degrees
- moved L109 259.6 mm to (77.9, -77.2), turned to 270 degrees
- moved L110 259.5 mm to (86.5, -77.2), turned to 270 degrees
- moved L77 243.8 mm to (86.5, -51.4), turned to 270 degrees
- moved L103 234.4 mm to (26.0, -77.2), turned to 270 degrees
- moved L104 234.3 mm to (34.6, -77.2), turned to 270 degrees
- moved L105 234.3 mm to (43.3, -77.2), turned to 270 degrees
- moved L93 234.2 mm to (34.6, -68.6), turned to 270 degrees
- moved L106 234.2 mm to (51.9, -77.2), turned to 270 degrees
- moved L94 234.1 mm to (43.3, -68.6), turned to 270 degrees
- moved L107 234.1 mm to (60.6, -77.2), turned to 270 degrees
- moved L95 234.0 mm to (51.9, -68.6), turned to 270 degrees
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Connections:
- removed net INROW1: L1.4-DIN
- removed net N$12 (its old number): L112.4-DIN, L113.2-DOUT
- removed net N$25 (its old number): L111.4-DIN, L112.2-DOUT
- removed net N$26 (its old number): L111.2-DOUT, L114.4-DIN
- removed net OUTGES: L114.2-DOUT
- removed net OUTROW1: L11.2-DOUT, L12.4-DIN
- removed net OUTROW10: L110.2-DOUT, L113.4-DIN
- removed net OUTROW2: L22.2-DOUT, L23.4-DIN
- removed net OUTROW3: L33.2-DOUT, L34.4-DIN
- removed net OUTROW4: L44.2-DOUT, L45.4-DIN
- removed net OUTROW5: L55.2-DOUT, L56.4-DIN
- removed net OUTROW6: L66.2-DOUT, L67.4-DIN
- removed net OUTROW7: L77.2-DOUT, L78.4-DIN
- removed net OUTROW8: L88.2-DOUT, L89.4-DIN
- removed net OUTROW9: L100.4-DIN, L99.2-DOUT
- net +5V: no longer C111.1, C112.1, C113.1, C114.1, L111.1-VDD, L112.1-VDD, L113.1-VDD, L114.1-VDD
- net GND: no longer C111.2, C112.2, C113.2, C114.2, L111.3-GND, L112.3-GND, L113.3-GND, L114.3-GND
Routing:
- net +5V: track 0.00 -> 1913.7 mm
- net GND: track 69.5 -> 1304.5 mm
- net N$64: track 0.00 -> 8.71 mm
- net N$94: track 0.00 -> 8.71 mm
- net N$44: track 0.00 -> 8.71 mm
- net N$34: track 0.00 -> 8.71 mm
- net N$74: track 0.00 -> 8.71 mm
- net N$24: track 0.00 -> 8.71 mm
- net N$54: track 0.00 -> 8.71 mm
- net N$12: track 0.00 -> 8.71 mm
- net N$84: track 0.00 -> 8.71 mm
- net N$63: track 0.00 -> 8.69 mm
- net N$43: track 0.00 -> 8.69 mm
- net N$33: track 0.00 -> 8.69 mm
- net N$93: track 0.00 -> 8.69 mm
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Other:
- board outline removed

Commit message: Eagle Layout geroutet
Parts:
- added C111, C112, C113, C114, C115: 100n, rcl:C1310
- added C116, C117: (no value), rcl:C0805
- added IC1: MEGA8-P, atmel:DIL28-3
- added LED1, LED2, LED3, LED4, LED5: (no value), led:CHIPLED_1206
- added Q2: (no value), crystal:HC49/S
- added R1, R2: (no value), rcl:M0805
- added R10, R11, R12, R3, R4, R5, R6, R7, R8, R9: (no value), rcl:M1206
- added S1, S2, S3, S4, S5: (no value), switch-omron:B3F-10XX
- added SG1: F/HMB, buzzer:F/HMB
- added SV1: (no value), con-harting-ml:ML6L
- moved S+1 118.7 mm to (-13.9, 84.8)
- moved C1 113.4 mm to (28.6, 112.3)
- moved C10 113.4 mm to (106.4, 112.3)
- moved C11 113.4 mm to (115.1, 112.3)
- moved C2 113.4 mm to (37.2, 112.3)
- moved C3 113.4 mm to (45.9, 112.3)
- moved C4 113.4 mm to (54.5, 112.3)
- moved C5 113.4 mm to (63.2, 112.3)
- moved C6 113.4 mm to (71.8, 112.3)
- moved C7 113.4 mm to (80.5, 112.3)
- moved C8 113.4 mm to (89.1, 112.3)
- moved C9 113.4 mm to (97.8, 112.3)
- moved L1 113.4 mm to (24.2, 110.8)
- moved L10 113.4 mm to (102.1, 110.8)
- moved L11 113.4 mm to (110.8, 110.8)
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Connections:
- removed net VCC: U$1.1
- new net INTA: R1.1, S+1.3
- new net INTB: R2.1, S+1.7
- new net LEDALARM: LED5.C
- new net LEDMIN1: IC1.16, LED1.C
- new net LEDMIN2: IC1.17, LED2.C, SV1.4
- new net LEDMIN3: IC1.18, LED3.C, SV1.1
- new net LEDMIN4: IC1.19, LED4.C, SV1.3
- new net N$103: L11.2-DOUT, L12.4-DIN
- new net N$104: L22.2-DOUT, L23.4-DIN
- new net N$105: L33.2-DOUT, L34.4-DIN
- new net N$106: L44.2-DOUT, L45.4-DIN
- new net N$107: L55.2-DOUT, L56.4-DIN
- new net N$108: L66.2-DOUT, L67.4-DIN
- new net N$109: L77.2-DOUT, L78.4-DIN
- new net N$110: L88.2-DOUT, L89.4-DIN
- new net N$111: L100.4-DIN, L99.2-DOUT
- new net N$112: C115.1, R8.1, S5.1
- new net N$113: C111.1, R9.1, S1.1
- new net N$114: LED1.A, R3.2
- new net N$115: LED2.A, R4.2
- new net N$116: LED3.A, R5.2
- new net N$117: LED4.A, R6.2
- new net N$118: LED5.A, R7.2
- new net N$119: IC1.27
- new net N$120: IC1.28
- new net N$121: IC1.4
- new net N$122: IC1.5
- new net N$123: C112.1, R10.1, S2.1
- new net N$124: C113.1, R11.1, S3.1
- new net N$125: C114.1, R12.1, S4.1
- new net N$126: IC1.23
- new net N$127: IC1.24
- new net N$128: IC1.25
- new net N$129: IC1.26
- new net N$130: IC1.2
- new net N$131: IC1.3
- new net N$132: IC1.6
- new net N$133: IC1.11
- new net N$134: IC1.12
- new net N$135: IC1.13
- new net N$136: C117.2, IC1.9, Q2.2
- new net N$137: C116.2, IC1.10, Q2.1
- new net N$141: IC1.15
- new net N$142: IC1.14
- new net RESET: IC1.1, SV1.5
- new net SCHALTER1: R9.2
- new net SCHALTER2: R10.2
- new net SCHALTER3: R11.2
- new net SCHALTER4: R12.2
- new net SCHALTER5: R8.2
- new net SCL: S+1.6
- new net SDA: S+1.5
- net +5V: now also IC1.20, IC1.21, IC1.7, R1.2, R2.2, R3.1, R4.1, R5.1, R6.1, R7.1, S+1.8, SV1.2, U$1.1
- net GND: now also C111.2, C112.2, C113.2, C114.2, C115.2, C116.1, C117.1, IC1.22, IC1.8, S1.3, S2.3, S3.3, S4.3, S5.3, SV1.6
Routing:
- net N$111: track 0.00 -> 92.8 mm
- net N$110: track 0.00 -> 92.6 mm
- net N$106: track 0.00 -> 92.6 mm
- net N$103: track 0.00 -> 92.5 mm
- net N$105: track 0.00 -> 92.5 mm
- net N$108: track 0.00 -> 92.5 mm
- net N$104: track 0.00 -> 92.5 mm
- net N$107: track 0.00 -> 92.5 mm
- net N$109: track 0.00 -> 92.5 mm
Other:
- board outline added: 130 x 130 mm

Commit message: Eagle VDD gelayoutet und vieles mehr
Parts:
- removed R3, R5, R6, R7: (no value), rcl:M1206
- removed SG1: F/HMB, buzzer:F/HMB
- added C118, C119, C120: 100n, rcl:C0805
- added L111: 10u, rcl:L2012C
- added LDR, R_LED1, R_LED2, R_LED3, R_LED4, R_LED5, R_LEDAL: (no value), rcl:M1206
- added PAD1, PAD2: (no value), wirepad:2,54/1,1
- added Q3: SUP75N06-08, transistor-fet:TO220
- added SP1: AL11P, buzzer:AL11P
- Q1: device special:Q -> crystal:HC49/S
- moved SV1 262.6 mm to (-11.6, 81.3), flipped to the bottom, turned to 270 degrees
- moved C111 248.7 mm to (58.1, 116.3), turned to 270 degrees
- moved R9 248.3 mm to (60.8, 118.4), turned to 270 degrees
- moved C116 223.2 mm to (-57.4, 67.9)
- moved C117 223.2 mm to (-57.4, 64.0)
- moved C114 210.3 mm to (67.9, 18.5), turned to 90 degrees
- moved S4 209.6 mm to (77.5, 17.0), flipped to the bottom, turned to 180 degrees
- moved R12 206.0 mm to (70.9, 15.9), turned to 90 degrees
- moved R8 197.9 mm to (91.0, 15.9), turned to 90 degrees
- moved C115 194.7 mm to (88.1, 18.5), turned to 90 degrees
- moved Q2 193.1 mm to (-23.8, 36.0)
- moved S5 187.8 mm to (97.5, 17.0), flipped to the bottom, turned to 180 degrees
- moved C113 186.0 mm to (48.3, 18.6), turned to 90 degrees
- moved S3 184.8 mm to (57.5, 17.0), flipped to the bottom, turned to 180 degrees
- moved R11 177.9 mm to (51.0, 16.1), turned to 90 degrees
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Connections:
- removed net N$124: C113.1, R11.1, S3.1
- removed net N$125: C114.1, R12.1, S4.1
- removed net N$128: IC1.25
- removed net N$129: IC1.26
- removed net N$130: IC1.2
- removed net N$131: IC1.3
- removed net N$132: IC1.6
- removed net N$133: IC1.11
- removed net N$134: IC1.12
- removed net N$135: IC1.13
- removed net N$141: IC1.15
- removed net N$142: IC1.14
- new net LDR: IC1.26, LDR.1, R4.2
- new net MATRIXIN: IC1.25, L1.4-DIN
- new net MATRIXOUT: L110.2-DOUT
- new net NC1: IC1.14, PAD1.1
- new net NC2: IC1.15, PAD2.1
- new net VDD: C1.1, C10.1, C100.1, C101.1, C102.1, C103.1, C104.1, C105.1, C106.1, C107.1, C108.1, C109.1, C11.1, C110.1, C12.1, C13.1, C14.1, C15.1, C16.1, C17.1, C18.1, C19.1, C2.1, C20.1, C21.1, C22.1, C23.1, C24.1, C25.1, C26.1, C27.1, C28.1, C29.1, C3.1, C30.1, C31.1, C32.1, C33.1, C34.1, C35.1, C36.1, C37.1, C38.1, C39.1, C4.1, C40.1, C41.1, C42.1, C43.1, C44.1, C45.1, C46.1, C47.1, C48.1, C49.1, C5.1, C50.1, C51.1, C52.1, C53.1, C54.1, C55.1, C56.1, C57.1, C58.1, C59.1, C6.1, C60.1, C61.1, C62.1, C63.1, C64.1, C65.1, C66.1, C67.1, C68.1, C69.1, C7.1, C70.1, C71.1, C72.1, C73.1, C74.1, C75.1, C76.1, C77.1, C78.1, C79.1, C8.1, C80.1, C81.1, C82.1, C83.1, C84.1, C85.1, C86.1, C87.1, C88.1, C89.1, C9.1, C90.1, C91.1, C92.1, C93.1, C94.1, C95.1, C96.1, C97.1, C98.1, C99.1, L1.1-VDD, L10.1-VDD, L100.1-VDD, L101.1-VDD, L102.1-VDD, L103.1-VDD, L104.1-VDD, L105.1-VDD, L106.1-VDD, L107.1-VDD, L108.1-VDD, L109.1-VDD, L11.1-VDD, L110.1-VDD, L12.1-VDD, L13.1-VDD, L14.1-VDD, L15.1-VDD, L16.1-VDD, L17.1-VDD, L18.1-VDD, L19.1-VDD, L2.1-VDD, L20.1-VDD, L21.1-VDD, L22.1-VDD, L23.1-VDD, L24.1-VDD, L25.1-VDD, L26.1-VDD, L27.1-VDD, L28.1-VDD, L29.1-VDD, L3.1-VDD, L30.1-VDD, L31.1-VDD, L32.1-VDD, L33.1-VDD, L34.1-VDD, L35.1-VDD, L36.1-VDD, L37.1-VDD, L38.1-VDD, L39.1-VDD, L4.1-VDD, L40.1-VDD, L41.1-VDD, L42.1-VDD, L43.1-VDD, L44.1-VDD, L45.1-VDD, L46.1-VDD, L47.1-VDD, L48.1-VDD, L49.1-VDD, L5.1-VDD, L50.1-VDD, L51.1-VDD, L52.1-VDD, L53.1-VDD, L54.1-VDD, L55.1-VDD, L56.1-VDD, L57.1-VDD, L58.1-VDD, L59.1-VDD, L6.1-VDD, L60.1-VDD, L61.1-VDD, L62.1-VDD, L63.1-VDD, L64.1-VDD, L65.1-VDD, L66.1-VDD, L67.1-VDD, L68.1-VDD, L69.1-VDD, L7.1-VDD, L70.1-VDD, L71.1-VDD, L72.1-VDD, L73.1-VDD, L74.1-VDD, L75.1-VDD, L76.1-VDD, L77.1-VDD, L78.1-VDD, L79.1-VDD, L8.1-VDD, L80.1-VDD, L81.1-VDD, L82.1-VDD, L83.1-VDD, L84.1-VDD, L85.1-VDD, L86.1-VDD, L87.1-VDD, L88.1-VDD, L89.1-VDD, L9.1-VDD, L90.1-VDD, L91.1-VDD, L92.1-VDD, L93.1-VDD, L94.1-VDD, L95.1-VDD, L96.1-VDD, L97.1-VDD, L98.1-VDD, L99.1-VDD, Q3.3
- net +5V: now also C120.2, L111.1, LDR.2, Q3.2, R_LED1.1, R_LED2.1, R_LED3.1, R_LED4.1, R_LED5.2, R_LEDAL.1, SP1.+; no longer C1.1, C10.1, C100.1, C101.1, C102.1, C103.1, C104.1, C105.1, C106.1, C107.1, C108.1, C109.1, C11.1, C110.1, C12.1, C13.1, C14.1, C15.1, C16.1, C17.1, C18.1, C19.1, C2.1, C20.1, C21.1, C22.1, C23.1, C24.1, C25.1, C26.1, C27.1, C28.1, C29.1, C3.1, C30.1, C31.1, C32.1, C33.1, C34.1, C35.1, C36.1, C37.1, C38.1, C39.1, C4.1, C40.1, C41.1, C42.1, C43.1, C44.1, C45.1, C46.1, C47.1, C48.1, C49.1, C5.1, C50.1, C51.1, C52.1, C53.1, C54.1, C55.1, C56.1, C57.1, C58.1, C59.1, C6.1, C60.1, C61.1, C62.1, C63.1, C64.1, C65.1, C66.1, C67.1, C68.1, C69.1, C7.1, C70.1, C71.1, C72.1, C73.1, C74.1, C75.1, C76.1, C77.1, C78.1, C79.1, C8.1, C80.1, C81.1, C82.1, C83.1, C84.1, C85.1, C86.1, C87.1, C88.1, C89.1, C9.1, C90.1, C91.1, C92.1, C93.1, C94.1, C95.1, C96.1, C97.1, C98.1, C99.1, IC1.20, IC1.21, L1.1-VDD, L10.1-VDD, L100.1-VDD, L101.1-VDD, L102.1-VDD, L103.1-VDD, L104.1-VDD, L105.1-VDD, L106.1-VDD, L107.1-VDD, L108.1-VDD, L109.1-VDD, L11.1-VDD, L110.1-VDD, L12.1-VDD, L13.1-VDD, L14.1-VDD, L15.1-VDD, L16.1-VDD, L17.1-VDD, L18.1-VDD, L19.1-VDD, L2.1-VDD, L20.1-VDD, L21.1-VDD, L22.1-VDD, L23.1-VDD, L24.1-VDD, L25.1-VDD, L26.1-VDD, L27.1-VDD, L28.1-VDD, L29.1-VDD, L3.1-VDD, L30.1-VDD, L31.1-VDD, L32.1-VDD, L33.1-VDD, L34.1-VDD, L35.1-VDD, L36.1-VDD, L37.1-VDD, L38.1-VDD, L39.1-VDD, L4.1-VDD, L40.1-VDD, L41.1-VDD, L42.1-VDD, L43.1-VDD, L44.1-VDD, L45.1-VDD, L46.1-VDD, L47.1-VDD, L48.1-VDD, L49.1-VDD, L5.1-VDD, L50.1-VDD, L51.1-VDD, L52.1-VDD, L53.1-VDD, L54.1-VDD, L55.1-VDD, L56.1-VDD, L57.1-VDD, L58.1-VDD, L59.1-VDD, L6.1-VDD, L60.1-VDD, L61.1-VDD, L62.1-VDD, L63.1-VDD, L64.1-VDD, L65.1-VDD, L66.1-VDD, L67.1-VDD, L68.1-VDD, L69.1-VDD, L7.1-VDD, L70.1-VDD, L71.1-VDD, L72.1-VDD, L73.1-VDD, L74.1-VDD, L75.1-VDD, L76.1-VDD, L77.1-VDD, L78.1-VDD, L79.1-VDD, L8.1-VDD, L80.1-VDD, L81.1-VDD, L82.1-VDD, L83.1-VDD, L84.1-VDD, L85.1-VDD, L86.1-VDD, L87.1-VDD, L88.1-VDD, L89.1-VDD, L9.1-VDD, L90.1-VDD, L91.1-VDD, L92.1-VDD, L93.1-VDD, L94.1-VDD, L95.1-VDD, L96.1-VDD, L97.1-VDD, L98.1-VDD, L99.1-VDD, R3.1, R4.1, R5.1, R6.1, R7.1
- net GND: now also C118.1, C119.1, C120.1, R4.1, S1.4, S2.4, S3.4, S4.4, S5.4
- net INTA: now also IC1.4
- net INTB: now also IC1.5
- net LEDALARM: now also IC1.23
- net N$112: now also IC1.2, SP1.-; no longer C115.1, R8.1, S5.1
- net N$113: now also C118.2, IC1.20, L111.2; no longer C111.1, R9.1, S1.1
- net N$114: now also R_LED1.2; no longer R3.2
- net N$115: now also R_LED2.2; no longer R4.2
- net N$116: now also R_LED3.2; no longer R5.2
- net N$117: now also R_LED4.2; no longer R6.2
- net N$118: now also R_LEDAL.2; no longer R7.2
- net N$119: now also R9.1, S1.1, S1.2; no longer IC1.27
- net N$120: now also R10.1, S2.1; no longer IC1.28
- net N$121: now also R11.1, S3.1; no longer IC1.4
- net N$122: now also R12.1, S4.1; no longer IC1.5
- net N$123: now also C119.2, IC1.21; no longer C112.1, R10.1, S2.1
- net N$126: now also R8.1, S5.1; no longer IC1.23
- net N$127: now also Q3.1
- net N$136: now also Q2.1; no longer Q2.2
- net N$137: now also Q2.2; no longer Q2.1
- net RESET: now also R_LED5.1
- net SCHALTER1: now also C111.1, IC1.3
- net SCHALTER2: now also C112.1, IC1.6
- net SCHALTER3: now also C113.1, IC1.11
- net SCHALTER4: now also C114.1, IC1.12
- net SCHALTER5: now also C115.1, IC1.13
- net SCL: now also IC1.28
- net SDA: now also IC1.27
Routing:
- net VDD: track 0.00 -> 1929.7 mm
- net +5V: track 1913.7 -> 244.0 mm
- net GND: track 1304.5 -> 1683.2 mm
- net LEDMIN1: track 0.00 -> 118.1 mm
- net LEDMIN2: track 0.00 -> 109.7 mm
- net N$127: track 0.00 -> 109.7 mm
- net LEDALARM: track 0.00 -> 46.6 mm
- net N$112: track 0.00 -> 43.5 mm
- net SCHALTER1: track 0.00 -> 38.5 mm
- net N$21: track 0.00 -> 16.4 mm
- net N$115: track 0.00 -> 11.1 mm
- net N$20: track 0.00 -> 11.0 mm
- net N$119: track 0.00 -> 10.5 mm
- net N$120: track 0.00 -> 3.70 mm
- net N$122: track 0.00 -> 3.33 mm
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