File: Eagle/Wordclock/Wordclock.brd (EAGLE design)
At the start: 130 x 130 mm, 281 parts, among them IC1 MEGA8-P, Q3 SUP75N06-08

Commit message: Bauteilliste exportiert
Parts:
- R_LED1, R_LED2, R_LED3, R_LED4, R_LEDAL: value (none) -> 120
- R_PHOTO: value (none) -> 49,9k
Changed lines of the file:
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@@
 <element name="PULLUP_INTA" library="rcl" package="R1206" value="4,7k" x="19.805" y="70.37" rot="R270"/>
 <element name="PULLUP_INTB" library="rcl" package="R1206" value="4,7k" x="42.98" y="121.535"/>
-<element name="R_LED1" library="rcl" package="M1206" value="" x="124.87" y="119.33" rot="R180"/>
-<element name="R_LED2" library="rcl" package="M1206" value="" x="120.16" y="23.7" rot="R270"/>
-<element name="R_LED3" library="rcl" package="M1206" value="" x="13.95" y="11.45" rot="R270"/>
-<element name="R_LED4" library="rcl" package="M1206" value="" x="33.07" y="125.31" rot="R180"/>
+<element name="R_LED1" library="rcl" package="M1206" value="120" x="124.87" y="119.33" rot="R180"/>
+<element name="R_LED2" library="rcl" package="M1206" value="120" x="120.16" y="23.7" rot="R270"/>
+<element name="R_LED3" library="rcl" package="M1206" value="120" x="13.95" y="11.45" rot="R270"/>
+<element name="R_LED4" library="rcl" package="M1206" value="120" x="33.07" y="125.31" rot="R180"/>
 <element name="LED1" library="led" package="CHIPLED_1206" value="" x="123.5" y="123.5"/>
 <element name="LED2" library="led" package="CHIPLED_1206" value="" x="123.5" y="11.5" rot="R180"/>
@@
 <element name="LED4" library="led" package="CHIPLED_1206" value="" x="11.5" y="123.5" rot="R180"/>
 <element name="LEDAL" library="led" package="CHIPLED_1206" value="" x="67.5" y="123.5"/>
-<element name="R_LEDAL" library="rcl" package="M1206" value="" x="70.82" y="121.81" rot="R180"/>
+<element name="R_LEDAL" library="rcl" package="M1206" value="120" x="70.82" y="121.81" rot="R180"/>
 <element name="IC1" library="atmel" package="DIL28-3" value="MEGA8-P" x="11.5" y="65" rot="MR270">
 <attribute name="OC_NEWARK" value="unknown" x="11.5" y="65" size="1.778" layer="28" rot="MR270" display="off"/>
@@
 <element name="Q3" library="transistor-fet" package="TO220" value="SUP75N06-08" x="124.17" y="108.27" rot="MR180"/>
 <element name="LDR" library="rcl" package="0204/5" value="" x="67.5" y="125" rot="MR180"/>
-<element name="R_PHOTO" library="rcl" package="M1206" value="" x="60.68" y="126.49" rot="R270"/>
+<element name="R_PHOTO" library="rcl" package="M1206" value="49,9k" x="60.68" y="126.49" rot="R270"/>
 <element name="PAD1" library="wirepad" package="2,54/1,1" value="" x="15.01" y="92"/>
 <element name="PAD2" library="wirepad" package="2,54/1,1" value="" x="15" y="101"/>

Commit message: Bestellung bei Reichelt und WS2812 und Kondensator auf 15p geändert
Bestellung bei Reichelt und WS2812 und Wert des Kondensator am AVR
Quarz auf 15p geändert
Parts:
- C116, C117: value 18p -> 15p
Changed lines of the file:
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@@
 <element name="C_S4" library="rcl" package="C1206" value="100n" x="66.75" y="17.84" rot="R90"/>
 <element name="R_S4" library="rcl" package="M1206" value="1k" x="70.3" y="15.14" rot="R180"/>
-<element name="C116" library="rcl" package="C0805" value="18p" x="20.94" y="59.64" rot="R270"/>
-<element name="C117" library="rcl" package="C0805" value="18p" x="17.86" y="63.06" rot="R270"/>
+<element name="C116" library="rcl" package="C0805" value="15p" x="20.94" y="59.64" rot="R270"/>
+<element name="C117" library="rcl" package="C0805" value="15p" x="17.86" y="63.06" rot="R270"/>
 <element name="SV1" library="con-harting-ml" package="ML6L" value="" x="11.46" y="37.02" rot="MR180">
 <attribute name="OC_NEWARK" value="unknown" x="11.46" y="37.02" size="1.778" layer="28" rot="MR180" display="off"/>
