File: Eagle/Wordclock/Wordclock.sch (EAGLE design)
At the start: 74 parts, among them IC1 74HC595D, IC2 74HC595D, IC3 74HC595D, IC4 74HC595D, IC5 74HC595D, IC6 74HC595D, IC7 74HC595D, IC8 74HC595D

Commit message: Eagle Adafruit added
Parts:
- added LED65, LED66, LED67, LED68: WS2812B, WS2812B:WS2812B
- added Q1: (no value), special:XTAL
Connections:
- new net N$82: Q1.1, S+1.X1
- new net N$83: Q1.2, S+1.X2
- new net N$85: LED65.DO, LED66.DI
- new net N$86: LED66.DO, LED67.DI
- new net N$87: LED67.DO, LED68.DI
- net N$81: now also S+1.GND
Other:
- note removed: "+5V"
- note removed: "GND"
Changed lines of the file:
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@@
 <layer number="54" name="bGND_GNDA" color="1" fill="9" visible="no" active="no"/>
 <layer number="56" name="wert" color="7" fill="1" visible="no" active="no"/>
+<layer number="57" name="tCAD" color="7" fill="1" visible="no" active="no"/>
 <layer number="90" name="Modules" color="5" fill="1" visible="yes" active="yes"/>
 <layer number="91" name="Nets" color="2" fill="1" visible="yes" active="yes"/>
@@
 <layer number="109" name="fp9" color="7" fill="1" visible="yes" active="yes"/>
 <layer number="110" name="fp0" color="7" fill="1" visible="yes" active="yes"/>
+<layer number="111" name="LPC17xx" color="7" fill="1" visible="yes" active="yes"/>
+<layer number="112" name="tSilk" color="7" fill="1" visible="yes" active="yes"/>
 <layer number="116" name="Patch_BOT" color="9" fill="4" visible="yes" active="yes"/>
 <layer number="121" name="_tsilk" color="7" fill="1" visible="yes" active="yes"/>
@@
 <layer number="123" name="tTestmark" color="7" fill="1" visible="yes" active="yes"/>
 <layer number="124" name="bTestmark" color="7" fill="1" visible="yes" active="yes"/>
+<layer number="125" name="_tNames" color="7" fill="1" visible="yes" active="yes"/>
+<layer number="126" name="_bNames" color="7" fill="1" visible="yes" active="yes"/>
+<layer number="127" name="_tValues" color="7" fill="1" visible="yes" active="yes"/>
+<layer number="128" name="_bValues" color="7" fill="1" visible="yes" active="yes"/>
 <layer number="131" name="tAdjust" color="7" fill="1" visible="yes" active="yes"/>
 <layer number="132" name="bAdjust" color="7" fill="1" visible="yes" active="yes"/>
 <layer number="144" name="Drill_legend" color="7" fill="1" visible="yes" active="yes"/>
+<layer number="150" name="Notes" color="7" fill="1" visible="no" active="yes"/>
 <layer number="151" name="HeatSink" color="7" fill="1" visible="yes" active="yes"/>
+<layer number="152" name="_bDocu" color="7" fill="1" visible="yes" active="yes"/>
+<layer number="153" name="FabDoc1" color="6" fill="1" visible="no" active="no"/>
+<layer number="154" name="FabDoc2" color="2" fill="1" visible="no" active="no"/>
+<layer number="155" name="FabDoc3" color="7" fill="15" visible="no" active="no"/>
 <layer number="199" name="Contour" color="7" fill="1" visible="yes" active="yes"/>
 <layer number="200" name="200bmp" color="1" fill="10" visible="no" active="no"/>
@@
 <layer number="215" name="215bmp" color="7" fill="1" visible="yes" active="yes"/>
 <layer number="216" name="216bmp" color="7" fill="1" visible="yes" active="yes"/>
+<layer number="217" name="217bmp" color="18" fill="1" visible="no" active="no"/>
+<layer number="218" name="218bmp" color="19" fill="1" visible="no" active="no"/>
+<layer number="219" name="219bmp" color="20" fill="1" visible="no" active="no"/>
+<layer number="220" name="220bmp" color="21" fill="1" visible="no" active="no"/>
+<layer number="221" name="221bmp" color="22" fill="1" visible="no" active="no"/>
+<layer number="222" name="222bmp" color="23" fill="1" visible="no" active="no"/>
+<layer number="223" name="223bmp" color="24" fill="1" visible="no" active="no"/>
+<layer number="224" name="224bmp" color="25" fill="1" visible="no" active="no"/>
+<layer number="248" name="Housing" color="7" fill="1" visible="yes" active="yes"/>
+<layer number="249" name="Edge" color="7" fill="1" visible="yes" active="yes"/>
 <layer number="250" name="Descript" color="7" fill="1" visible="no" active="no"/>
 <layer number="251" name="SMDround" color="7" fill="1" visible="no" active="no"/>
@@
 <part name="S+1" library="eagle-library-edeca.net-v5" deviceset="DS1337" device="+"/>
 <part name="U$1" library="eagle-library-edeca.net-v5" deviceset="MINI-USB" device=""/>
+<part name="Q1" library="special" deviceset="XTAL" device=""/>
+<part name="LED65" library="WS2812B" deviceset="WS2812B" device=""/>
+<part name="LED66" library="WS2812B" deviceset="WS2812B" device=""/>
+<part name="LED67" library="WS2812B" deviceset="WS2812B" device=""/>
+<part name="LED68" library="WS2812B" deviceset="WS2812B" device=""/>
 </parts>
 <sheets>
 <sheet>
 <plain>
-<text x="-50.8" y="106.68" size="1.778" layer="91">+5V</text>
-<text x="-48.26" y="63.5" size="1.778" layer="91">GND</text>
 </plain>
 <instances>
@@
 <instance part="S+1" gate="G$1" x="-55.88" y="50.8"/>
 <instance part="U$1" gate="G$1" x="-53.34" y="78.74"/>
+<instance part="Q1" gate="G$1" x="-86.36" y="53.34"/>
+<instance part="LED65" gate="G$1" x="-93.98" y="10.16"/>
+<instance part="LED66" gate="G$1" x="-68.58" y="10.16"/>
+<instance part="LED67" gate="G$1" x="-43.18" y="10.16"/>
+<instance part="LED68" gate="G$1" x="-17.78" y="10.16"/>
 </instances>
 <busses>
@@
 <wire x1="-58.42" y1="73.66" x2="-58.42" y2="60.96" width="0.1524" layer="91"/>
 <wire x1="-58.42" y1="60.96" x2="-38.1" y2="60.96" width="0.1524" layer="91"/>
-</segment>
-</net>
+<wire x1="-38.1" y1="35.56" x2="-38.1" y2="60.96" width="0.1524" layer="91"/>
+<pinref part="S+1" gate="G$1" pin="GND"/>
+<wire x1="-68.58" y1="45.72" x2="-68.58" y2="35.56" width="0.1524" layer="91"/>
+<wire x1="-68.58" y1="35.56" x2="-38.1" y2="35.56" width="0.1524" layer="91"/>
+</segment>
+</net>
+<net name="N$82" class="0">
+<segment>
+<pinref part="Q1" gate="G$1" pin="1"/>
+<wire x1="-91.44" y1="53.34" x2="-91.44" y2="58.42" width="0.1524" layer="91"/>
+<pinref part="S+1" gate="G$1" pin="X1"/>
+<wire x1="-91.44" y1="58.42" x2="-68.58" y2="58.42" width="0.1524" layer="91"/>
+<wire x1="-68.58" y1="58.42" x2="-68.58" y2="53.34" width="0.1524" layer="91"/>
+</segment>
+</net>
+<net name="N$83" class="0">
+<segment>
+<pinref part="Q1" gate="G$1" pin="2"/>
+<wire x1="-81.28" y1="53.34" x2="-73.66" y2="53.34" width="0.1524" layer="91"/>
+<wire x1="-73.66" y1="53.34" x2="-73.66" y2="50.8" width="0.1524" layer="91"/>
+<pinref part="S+1" gate="G$1" pin="X2"/>
+<wire x1="-73.66" y1="50.8" x2="-68.58" y2="50.8" width="0.1524" layer="91"/>
+</segment>
+</net>
+<net name="N$85" class="0">
+<segment>
+<pinref part="LED65" gate="G$1" pin="DO"/>
+<pinref part="LED66" gate="G$1" pin="DI"/>
+</segment>
+</net>
+<net name="N$86" class="0">
+<segment>
+<pinref part="LED66" gate="G$1" pin="DO"/>
+<pinref part="LED67" gate="G$1" pin="DI"/>
+</segment>
+</net>
+<net name="N$87" class="0">
+<segment>
+<pinref part="LED67" gate="G$1" pin="DO"/>
+<pinref part="LED68" gate="G$1" pin="DI"/>
+</segment>
+</net>

Commit message: Eagle Fehler verbessert
Parts:
- removed IC2, IC3, IC4, IC5, IC6, IC7, IC8: 74HC595D, 74xx-eu:74HC595D
- removed LED10, LED11, LED12, LED13, LED14, LED15, LED16, LED17, LED18, LED19, LED20, LED21, LED22, LED23, LED24, LED25, LED26, LED27, LED28, LED29, LED30, LED31, LED32, LED33, LED34, LED35, LED36, LED37, LED38, LED39, LED40, LED41, LED42, LED43, LED44, LED45, LED46, LED47, LED48, LED49, LED50, LED51, LED52, LED53, LED54, LED55, LED56, LED57, LED58, LED59, LED60, LED61, LED62, LED63, LED64, LED9: (no value), led:LED3MM
- removed LED65, LED66, LED67, LED68: WS2812B, WS2812B:WS2812B
- added R1, R2, R3, R4, R5, R6, R7, R8: (no value), resistor:R-EU_MELF0102W
- LED1, LED2, LED3, LED4, LED5, LED6, LED7, LED8: device led:LED3MM -> led:LED
Connections:
- net N$81 renamed GND
- removed net N$20 (its old number): IC3A.QB, LED18.A
- removed net N$21 (its old number): IC3A.QC, LED19.A
- removed net N$22: IC3A.QE, LED21.A
- removed net N$23: IC3A.QD, LED20.A
- removed net N$24: IC3A.QF, LED22.A
- removed net N$25: IC3A.QG, LED23.A
- removed net N$26: IC3A.QH, LED24.A
- removed net N$27: LED17.C, LED18.C, LED19.C, LED20.C, LED21.C, LED22.C, LED23.C, LED24.C
- removed net N$28: IC4A.QA, LED25.A
- removed net N$29: IC4A.QB, LED26.A
- removed net N$30: IC4A.QC, LED27.A
- removed net N$31: IC4A.QE, LED29.A
- removed net N$32: IC4A.QD, LED28.A
- removed net N$33: IC4A.QF, LED30.A
- removed net N$34: IC4A.QG, LED31.A
- removed net N$35: IC4A.QH, LED32.A
- removed net N$36: LED25.C, LED26.C, LED27.C, LED28.C, LED29.C, LED30.C, LED31.C, LED32.C
- removed net N$37: IC5A.QA, LED33.A
- removed net N$38: IC5A.QB, LED34.A
- removed net N$39: IC5A.QC, LED35.A
- removed net N$40: IC5A.QE, LED37.A
- removed net N$41: IC5A.QD, LED36.A
- removed net N$42: IC5A.QF, LED38.A
- removed net N$43: IC5A.QG, LED39.A
- removed net N$44: IC5A.QH, LED40.A
- removed net N$45: LED33.C, LED34.C, LED35.C, LED36.C, LED37.C, LED38.C, LED39.C, LED40.C
- removed net N$46: IC6A.QA, LED41.A
- removed net N$47: IC6A.QB, LED42.A
- removed net N$48: IC6A.QC, LED43.A
- removed net N$49: IC6A.QE, LED45.A
- removed net N$50: IC6A.QD, LED44.A
- removed net N$51: IC6A.QF, LED46.A
- removed net N$52: IC6A.QG, LED47.A
- removed net N$53: IC6A.QH, LED48.A
- removed net N$54: LED41.C, LED42.C, LED43.C, LED44.C, LED45.C, LED46.C, LED47.C, LED48.C
- removed net N$55: IC7A.QA, LED49.A
- removed net N$56: IC7A.QB, LED50.A
- removed net N$57: IC7A.QC, LED51.A
- removed net N$58: IC7A.QE, LED53.A
- removed net N$59: IC7A.QD, LED52.A
- removed net N$60: IC7A.QF, LED54.A
- removed net N$61: IC7A.QG, LED55.A
- removed net N$62: IC7A.QH, LED56.A
- removed net N$63: LED49.C, LED50.C, LED51.C, LED52.C, LED53.C, LED54.C, LED55.C, LED56.C
- removed net N$64: IC8A.QA, LED57.A
- removed net N$65: IC8A.QB, LED58.A
- removed net N$66: IC8A.QC, LED59.A
- removed net N$67: IC8A.QE, LED61.A
- removed net N$68: IC8A.QD, LED60.A
- removed net N$69: IC8A.QF, LED62.A
- removed net N$70: IC8A.QG, LED63.A
- removed net N$71: IC8A.QH, LED64.A
- removed net N$72: LED57.C, LED58.C, LED59.C, LED60.C, LED61.C, LED62.C, LED63.C, LED64.C
- removed net N$73: IC5A.QH*, IC6A.SER
- removed net N$74: IC6A.QH*, IC7A.SER
- removed net N$75: IC7A.QH*, IC8A.SER
- removed net N$76: IC1A.SER, IC8A.QH*
- removed net N$77: IC1A.QH*, IC2A.SER
- removed net N$78: IC2A.QH*, IC3A.SER
- removed net N$79: IC3A.QH*, IC4A.SER
- removed net N$80: U$1.1
- removed net N$85: LED65.DO, LED66.DI
- removed net N$86: LED66.DO, LED67.DI
- removed net N$87: LED67.DO, LED68.DI
- new net VCC: S+1.VCC, U$1.1
- net N$10: now also LED8.C, R8.1; no longer IC2A.QA, LED9.A
- net N$11: now also LED1.C, R1.1; no longer IC2A.QB, LED10.A
- net N$12: now also LED2.C, R2.1; no longer IC2A.QC, LED11.A
- net N$13: now also LED3.C, R3.1; no longer IC2A.QE, LED13.A
- net N$14: now also LED5.C, R5.1; no longer IC2A.QD, LED12.A
- net N$15: now also LED6.C, R6.1; no longer IC2A.QF, LED14.A
- net N$16: now also LED7.C, R7.1; no longer IC2A.QG, LED15.A
- net N$17: now also R1.2, R2.2, R3.2, R4.2, R5.2, R6.2, R7.2, R8.2; no longer IC2A.QH, LED16.A
- net N$18: now also IC1A.SER; no longer LED10.C, LED11.C, LED12.C, LED13.C, LED14.C, LED15.C, LED16.C, LED9.C
- net N$19: now also IC1A.QH*; no longer IC3A.QA, LED17.A
- net N$9: now also R4.1; no longer LED1.C, LED2.C, LED3.C, LED5.C, LED6.C, LED7.C, LED8.C
Other:
- moved on the sheet: IC1, LED1, LED2, LED3, LED4, LED5, LED6, LED7, LED8, Q1, U$1

Commit message: Eagle Änderung
Connections:
- removed net N$17: R1.2, R2.2, R3.2, R4.2, R5.2, R6.2, R7.2, R8.2
- net GND: now also R1.2, R2.2, R3.2, R4.2, R5.2, R6.2, R7.2, R8.2
Changed lines of the file:
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@@
-</segment>
-</net>
-<net name="N$17" class="0">
-<segment>
-<pinref part="R8" gate="G$1" pin="2"/>
-<wire x1="134.62" y1="99.06" x2="137.16" y2="99.06" width="0.1524" layer="91"/>
-<wire x1="137.16" y1="99.06" x2="137.16" y2="101.6" width="0.1524" layer="91"/>
-<pinref part="R1" gate="G$1" pin="2"/>
-<wire x1="137.16" y1="101.6" x2="137.16" y2="104.14" width="0.1524" layer="91"/>
-<wire x1="137.16" y1="104.14" x2="137.16" y2="106.68" width="0.1524" layer="91"/>
-<wire x1="137.16" y1="106.68" x2="137.16" y2="109.22" width="0.1524" layer="91"/>
-<wire x1="137.16" y1="109.22" x2="137.16" y2="111.76" width="0.1524" layer="91"/>
-<wire x1="137.16" y1="111.76" x2="137.16" y2="114.3" width="0.1524" layer="91"/>
-<wire x1="137.16" y1="114.3" x2="137.16" y2="116.84" width="0.1524" layer="91"/>
-<wire x1="137.16" y1="116.84" x2="134.62" y2="116.84" width="0.1524" layer="91"/>
-<pinref part="R2" gate="G$1" pin="2"/>
-<wire x1="134.62" y1="114.3" x2="137.16" y2="114.3" width="0.1524" layer="91"/>
-<junction x="137.16" y="114.3"/>
-<pinref part="R3" gate="G$1" pin="2"/>
-<wire x1="134.62" y1="111.76" x2="137.16" y2="111.76" width="0.1524" layer="91"/>
-<junction x="137.16" y="111.76"/>
-<pinref part="R4" gate="G$1" pin="2"/>
-<wire x1="134.62" y1="109.22" x2="137.16" y2="109.22" width="0.1524" layer="91"/>
-<junction x="137.16" y="109.22"/>
-<pinref part="R5" gate="G$1" pin="2"/>
-<wire x1="134.62" y1="106.68" x2="137.16" y2="106.68" width="0.1524" layer="91"/>
-<junction x="137.16" y="106.68"/>
-<pinref part="R6" gate="G$1" pin="2"/>
-<wire x1="134.62" y1="104.14" x2="137.16" y2="104.14" width="0.1524" layer="91"/>
-<junction x="137.16" y="104.14"/>
-<pinref part="R7" gate="G$1" pin="2"/>
-<wire x1="134.62" y1="101.6" x2="137.16" y2="101.6" width="0.1524" layer="91"/>
-<junction x="137.16" y="101.6"/>
 </segment>
 </net>
@@
 <label x="-71.12" y="45.72" size="1.778" layer="95" rot="R180" xref="yes"/>
 </segment>
+<segment>
+<pinref part="R8" gate="G$1" pin="2"/>
+<wire x1="134.62" y1="99.06" x2="137.16" y2="99.06" width="0.1524" layer="91"/>
+<wire x1="137.16" y1="99.06" x2="137.16" y2="101.6" width="0.1524" layer="91"/>
+<pinref part="R1" gate="G$1" pin="2"/>
+<wire x1="137.16" y1="101.6" x2="137.16" y2="104.14" width="0.1524" layer="91"/>
+<wire x1="137.16" y1="104.14" x2="137.16" y2="106.68" width="0.1524" layer="91"/>
+<wire x1="137.16" y1="106.68" x2="137.16" y2="109.22" width="0.1524" layer="91"/>
+<wire x1="137.16" y1="109.22" x2="137.16" y2="111.76" width="0.1524" layer="91"/>
+<wire x1="137.16" y1="111.76" x2="137.16" y2="114.3" width="0.1524" layer="91"/>
+<wire x1="137.16" y1="114.3" x2="137.16" y2="116.84" width="0.1524" layer="91"/>
+<wire x1="137.16" y1="116.84" x2="134.62" y2="116.84" width="0.1524" layer="91"/>
+<pinref part="R2" gate="G$1" pin="2"/>
+<wire x1="134.62" y1="114.3" x2="137.16" y2="114.3" width="0.1524" layer="91"/>
+<junction x="137.16" y="114.3"/>
+<pinref part="R3" gate="G$1" pin="2"/>
+<wire x1="134.62" y1="111.76" x2="137.16" y2="111.76" width="0.1524" layer="91"/>
+<junction x="137.16" y="111.76"/>
+<pinref part="R4" gate="G$1" pin="2"/>
+<wire x1="134.62" y1="109.22" x2="137.16" y2="109.22" width="0.1524" layer="91"/>
+<junction x="137.16" y="109.22"/>
+<pinref part="R5" gate="G$1" pin="2"/>
+<wire x1="134.62" y1="106.68" x2="137.16" y2="106.68" width="0.1524" layer="91"/>
+<junction x="137.16" y="106.68"/>
+<pinref part="R6" gate="G$1" pin="2"/>
+<wire x1="134.62" y1="104.14" x2="137.16" y2="104.14" width="0.1524" layer="91"/>
+<junction x="137.16" y="104.14"/>
+<pinref part="R7" gate="G$1" pin="2"/>
+<wire x1="134.62" y1="101.6" x2="137.16" y2="101.6" width="0.1524" layer="91"/>
+<junction x="137.16" y="101.6"/>
+<label x="137.16" y="99.06" size="1.778" layer="95" xref="yes"/>
+</segment>
 </net>

Commit message: Eagel WS2812 added
Parts:
- removed IC1: 74HC595D, 74xx-eu:74HC595D
- removed LED1, LED2, LED3, LED4, LED5, LED6, LED7, LED8: (no value), led:LED
- removed R1, R2, R3, R4, R5, R6, R7, R8: (no value), resistor:R-EU_MELF0102W
- added C1, C10, C100, C101, C102, C103, C104, C105, C106, C107, C108, C109, C11, C110, C12, C13, C14, C15, C16, C17, C18, C19, C2, C20, C21, C22, C23, C24, C25, C26, C27, C28, C29, C3, C30, C31, C32, C33, C34, C35, C36, C37, C38, C39, C4, C40, C41, C42, C43, C44, C45, C46, C47, C48, C49, C5, C50, C51, C52, C53, C54, C55, C56, C57, C58, C59, C6, C60, C61, C62, C63, C64, C65, C66, C67, C68, C69, C7, C70, C71, C72, C73, C74, C75, C76, C77, C78, C79, C8, C80, C81, C82, C83, C84, C85, C86, C87, C88, C89, C9, C90, C91, C92, C93, C94, C95, C96, C97, C98, C99: 100n, rcl:C-EUC1310
- added L1, L10, L100, L101, L102, L103, L104, L105, L106, L107, L108, L109, L11, L110, L12, L13, L14, L15, L16, L17, L18, L19, L2, L20, L21, L22, L23, L24, L25, L26, L27, L28, L29, L3, L30, L31, L32, L33, L34, L35, L36, L37, L38, L39, L4, L40, L41, L42, L43, L44, L45, L46, L47, L48, L49, L5, L50, L51, L52, L53, L54, L55, L56, L57, L58, L59, L6, L60, L61, L62, L63, L64, L65, L66, L67, L68, L69, L7, L70, L71, L72, L73, L74, L75, L76, L77, L78, L79, L8, L80, L81, L82, L83, L84, L85, L86, L87, L88, L89, L9, L90, L91, L92, L93, L94, L95, L96, L97, L98, L99: WS2812B, adafruit:WS2812B
Connections:
- removed net N$11: LED1.C, R1.1
- new net +5V: C1.1, C10.1, C100.1, C101.1, C102.1, C103.1, C104.1, C105.1, C106.1, C107.1, C108.1, C109.1, C11.1, C110.1, C12.1, C13.1, C14.1, C15.1, C16.1, C17.1, C18.1, C19.1, C2.1, C20.1, C21.1, C22.1, C23.1, C24.1, C25.1, C26.1, C27.1, C28.1, C29.1, C3.1, C30.1, C31.1, C32.1, C33.1, C34.1, C35.1, C36.1, C37.1, C38.1, C39.1, C4.1, C40.1, C41.1, C42.1, C43.1, C44.1, C45.1, C46.1, C47.1, C48.1, C49.1, C5.1, C50.1, C51.1, C52.1, C53.1, C54.1, C55.1, C56.1, C57.1, C58.1, C59.1, C6.1, C60.1, C61.1, C62.1, C63.1, C64.1, C65.1, C66.1, C67.1, C68.1, C69.1, C7.1, C70.1, C71.1, C72.1, C73.1, C74.1, C75.1, C76.1, C77.1, C78.1, C79.1, C8.1, C80.1, C81.1, C82.1, C83.1, C84.1, C85.1, C86.1, C87.1, C88.1, C89.1, C9.1, C90.1, C91.1, C92.1, C93.1, C94.1, C95.1, C96.1, C97.1, C98.1, C99.1, L1.VDD, L10.VDD, L100.VDD, L101.VDD, L102.VDD, L103.VDD, L104.VDD, L105.VDD, L106.VDD, L107.VDD, L108.VDD, L109.VDD, L11.VDD, L110.VDD, L12.VDD, L13.VDD, L14.VDD, L15.VDD, L16.VDD, L17.VDD, L18.VDD, L19.VDD, L2.VDD, L20.VDD, L21.VDD, L22.VDD, L23.VDD, L24.VDD, L25.VDD, L26.VDD, L27.VDD, L28.VDD, L29.VDD, L3.VDD, L30.VDD, L31.VDD, L32.VDD, L33.VDD, L34.VDD, L35.VDD, L36.VDD, L37.VDD, L38.VDD, L39.VDD, L4.VDD, L40.VDD, L41.VDD, L42.VDD, L43.VDD, L44.VDD, L45.VDD, L46.VDD, L47.VDD, L48.VDD, L49.VDD, L5.VDD, L50.VDD, L51.VDD, L52.VDD, L53.VDD, L54.VDD, L55.VDD, L56.VDD, L57.VDD, L58.VDD, L59.VDD, L6.VDD, L60.VDD, L61.VDD, L62.VDD, L63.VDD, L64.VDD, L65.VDD, L66.VDD, L67.VDD, L68.VDD, L69.VDD, L7.VDD, L70.VDD, L71.VDD, L72.VDD, L73.VDD, L74.VDD, L75.VDD, L76.VDD, L77.VDD, L78.VDD, L79.VDD, L8.VDD, L80.VDD, L81.VDD, L82.VDD, L83.VDD, L84.VDD, L85.VDD, L86.VDD, L87.VDD, L88.VDD, L89.VDD, L9.VDD, L90.VDD, L91.VDD, L92.VDD, L93.VDD, L94.VDD, L95.VDD, L96.VDD, L97.VDD, L98.VDD, L99.VDD
- new net N$100: L90.DOUT, L91.DIN
- new net N$101: L91.DOUT, L92.DIN
- new net N$102: L92.DOUT, L93.DIN
- new net N$103: L93.DOUT, L94.DIN
- new net N$104: L94.DOUT, L95.DIN
- new net N$105: L95.DOUT, L96.DIN
- new net N$106: L96.DOUT, L97.DIN
- new net N$107: L97.DOUT, L98.DIN
- new net N$108: L98.DOUT, L99.DIN
- new net N$111: L100.DOUT, L101.DIN
- new net N$112: L101.DOUT, L102.DIN
- new net N$113: L102.DOUT, L103.DIN
- new net N$114: L103.DOUT, L104.DIN
- new net N$115: L104.DOUT, L105.DIN
- new net N$116: L105.DOUT, L106.DIN
- new net N$117: L106.DOUT, L107.DIN
- new net N$118: L107.DOUT, L108.DIN
- new net N$119: L108.DOUT, L109.DIN
- new net N$120: L109.DOUT, L110.DIN
- new net N$17: L16.DOUT, L17.DIN
- new net N$22: L19.DOUT, L20.DIN
- new net N$23: L20.DOUT, L21.DIN
- new net N$24: L21.DOUT, L22.DIN
- new net N$27: L23.DOUT, L24.DIN
- new net N$28: L24.DOUT, L25.DIN
- new net N$29: L25.DOUT, L26.DIN
- new net N$30: L26.DOUT, L27.DIN
- new net N$31: L27.DOUT, L28.DIN
- new net N$32: L28.DOUT, L29.DIN
- new net N$33: L29.DOUT, L30.DIN
- new net N$34: L30.DOUT, L31.DIN
- new net N$35: L31.DOUT, L32.DIN
- new net N$36: L32.DOUT, L33.DIN
- new net N$39: L34.DOUT, L35.DIN
- new net N$40: L35.DOUT, L36.DIN
- new net N$41: L36.DOUT, L37.DIN
- new net N$42: L37.DOUT, L38.DIN
- new net N$43: L38.DOUT, L39.DIN
- new net N$44: L39.DOUT, L40.DIN
- new net N$45: L40.DOUT, L41.DIN
- new net N$46: L41.DOUT, L42.DIN
- new net N$47: L42.DOUT, L43.DIN
- new net N$48: L43.DOUT, L44.DIN
- new net N$51: L45.DOUT, L46.DIN
- new net N$52: L46.DOUT, L47.DIN
- new net N$53: L47.DOUT, L48.DIN
- new net N$54: L48.DOUT, L49.DIN
- new net N$55: L49.DOUT, L50.DIN
- new net N$56: L50.DOUT, L51.DIN
- new net N$57: L51.DOUT, L52.DIN
- new net N$58: L52.DOUT, L53.DIN
- new net N$59: L53.DOUT, L54.DIN
- new net N$60: L54.DOUT, L55.DIN
- new net N$63: L56.DOUT, L57.DIN
- new net N$64: L57.DOUT, L58.DIN
- new net N$65: L58.DOUT, L59.DIN
- new net N$66: L59.DOUT, L60.DIN
- new net N$67: L60.DOUT, L61.DIN
- new net N$68: L61.DOUT, L62.DIN
- new net N$69: L62.DOUT, L63.DIN
- new net N$70: L63.DOUT, L64.DIN
- new net N$71: L64.DOUT, L65.DIN
- new net N$72: L65.DOUT, L66.DIN
- new net N$75: L67.DOUT, L68.DIN
- new net N$76: L68.DOUT, L69.DIN
- new net N$77: L69.DOUT, L70.DIN
- new net N$78: L70.DOUT, L71.DIN
- new net N$79: L71.DOUT, L72.DIN
- new net N$80: L72.DOUT, L73.DIN
- new net N$81: L73.DOUT, L74.DIN
- new net N$82: L74.DOUT, L75.DIN
- new net N$83: L75.DOUT, L76.DIN
- new net N$84: L76.DOUT, L77.DIN
- new net N$87: L78.DOUT, L79.DIN
- new net N$88: L79.DOUT, L80.DIN
- new net N$89: L80.DOUT, L81.DIN
- new net N$90: L81.DOUT, L82.DIN
- new net N$91: L82.DOUT, L83.DIN
- new net N$92: L83.DOUT, L84.DIN
- new net N$93: L84.DOUT, L85.DIN
- new net N$94: L85.DOUT, L86.DIN
- new net N$95: L86.DOUT, L87.DIN
- new net N$96: L87.DOUT, L88.DIN
- new net N$99: L89.DOUT, L90.DIN
- new net OUTROW1: L11.DOUT, L12.DIN
- new net OUTROW10: L110.DOUT
- new net OUTROW2: L22.DOUT, L23.DIN
- new net OUTROW3: L33.DOUT, L34.DIN
- new net OUTROW4: L44.DOUT, L45.DIN
- new net OUTROW5: L55.DOUT, L56.DIN
- new net OUTROW6: L66.DOUT, L67.DIN
- new net OUTROW7: L77.DOUT, L78.DIN
- new net OUTROW8: L88.DOUT, L89.DIN
- new net OUTROW9: L100.DIN, L99.DOUT
- net GND: now also C1.2, C10.2, C100.2, C101.2, C102.2, C103.2, C104.2, C105.2, C106.2, C107.2, C108.2, C109.2, C11.2, C110.2, C12.2, C13.2, C14.2, C15.2, C16.2, C17.2, C18.2, C19.2, C2.2, C20.2, C21.2, C22.2, C23.2, C24.2, C25.2, C26.2, C27.2, C28.2, C29.2, C3.2, C30.2, C31.2, C32.2, C33.2, C34.2, C35.2, C36.2, C37.2, C38.2, C39.2, C4.2, C40.2, C41.2, C42.2, C43.2, C44.2, C45.2, C46.2, C47.2, C48.2, C49.2, C5.2, C50.2, C51.2, C52.2, C53.2, C54.2, C55.2, C56.2, C57.2, C58.2, C59.2, C6.2, C60.2, C61.2, C62.2, C63.2, C64.2, C65.2, C66.2, C67.2, C68.2, C69.2, C7.2, C70.2, C71.2, C72.2, C73.2, C74.2, C75.2, C76.2, C77.2, C78.2, C79.2, C8.2, C80.2, C81.2, C82.2, C83.2, C84.2, C85.2, C86.2, C87.2, C88.2, C89.2, C9.2, C90.2, C91.2, C92.2, C93.2, C94.2, C95.2, C96.2, C97.2, C98.2, C99.2, L1.GND, L10.GND, L100.GND, L101.GND, L102.GND, L103.GND, L104.GND, L105.GND, L106.GND, L107.GND, L108.GND, L109.GND, L11.GND, L110.GND, L12.GND, L13.GND, L14.GND, L15.GND, L16.GND, L17.GND, L18.GND, L19.GND, L2.GND, L20.GND, L21.GND, L22.GND, L23.GND, L24.GND, L25.GND, L26.GND, L27.GND, L28.GND, L29.GND, L3.GND, L30.GND, L31.GND, L32.GND, L33.GND, L34.GND, L35.GND, L36.GND, L37.GND, L38.GND, L39.GND, L4.GND, L40.GND, L41.GND, L42.GND, L43.GND, L44.GND, L45.GND, L46.GND, L47.GND, L48.GND, L49.GND, L5.GND, L50.GND, L51.GND, L52.GND, L53.GND, L54.GND, L55.GND, L56.GND, L57.GND, L58.GND, L59.GND, L6.GND, L60.GND, L61.GND, L62.GND, L63.GND, L64.GND, L65.GND, L66.GND, L67.GND, L68.GND, L69.GND, L7.GND, L70.GND, L71.GND, L72.GND, L73.GND, L74.GND, L75.GND, L76.GND, L77.GND, L78.GND, L79.GND, L8.GND, L80.GND, L81.GND, L82.GND, L83.GND, L84.GND, L85.GND, L86.GND, L87.GND, L88.GND, L89.GND, L9.GND, L90.GND, L91.GND, L92.GND, L93.GND, L94.GND, L95.GND, L96.GND, L97.GND, L98.GND, L99.GND; no longer R1.2, R2.2, R3.2, R4.2, R5.2, R6.2, R7.2, R8.2
- net N$1: now also L1.DOUT, L2.DIN; no longer IC1A.QE, LED5.A
- net N$10: now also L10.DOUT, L11.DIN; no longer LED8.C, R8.1
- net N$12: now also L1.DIN; no longer LED2.C, R2.1
- net N$13: now also L12.DOUT, L13.DIN; no longer LED3.C, R3.1
- net N$14: now also L13.DOUT, L14.DIN; no longer LED5.C, R5.1
- net N$15: now also L14.DOUT, L15.DIN; no longer LED6.C, R6.1
- net N$16: now also L15.DOUT, L16.DIN; no longer LED7.C, R7.1
- net N$18: now also L17.DOUT, L18.DIN; no longer IC1A.SER
- net N$19: now also L18.DOUT, L19.DIN; no longer IC1A.QH*
- net N$2: now also L2.DOUT, L3.DIN; no longer IC1A.QF, LED6.A
- net N$3: now also L3.DOUT, L4.DIN; no longer IC1A.QG, LED7.A
- net N$4: now also L4.DOUT, L5.DIN; no longer IC1A.QH, LED8.A
- net N$5: now also L6.DOUT, L7.DIN; no longer IC1A.QD, LED4.A
- net N$6: now also L5.DOUT, L6.DIN; no longer IC1A.QC, LED3.A
- net N$7: now also L7.DOUT, L8.DIN; no longer IC1A.QB, LED2.A
- net N$8: now also L8.DOUT, L9.DIN; no longer IC1A.QA, LED1.A
- net N$9: now also L10.DIN, L9.DOUT; no longer LED4.C, R4.1
- net VCC: no longer S+1.VCC

Commit message: WS2812 Layout versucht
Parts:
- added C111, C112, C113, C114: 100n, rcl:C-EUC1310
- added L111, L112, L113, L114: WS2812B, adafruit:WS2812B
Connections:
- net N$12 renamed INROW1
- new net N$12: L112.DIN, L113.DOUT
- new net N$25: L111.DIN, L112.DOUT
- new net N$26: L111.DOUT, L114.DIN
- new net OUTGES: L114.DOUT
- net +5V: now also C111.1, C112.1, C113.1, C114.1, L111.VDD, L112.VDD, L113.VDD, L114.VDD
- net GND: now also C111.2, C112.2, C113.2, C114.2, L111.GND, L112.GND, L113.GND, L114.GND
- net OUTROW10: now also L113.DIN

Commit message: Wordclock Matrix gelayoutet
Matrix alle Zeilen einzeln gelautet, Zeilen sind noch nicht verbunden
Parts:
- removed C111, C112, C113, C114: 100n, rcl:C-EUC1310
- removed L111, L112, L113, L114: WS2812B, adafruit:WS2812B
Connections:
- removed net INROW1: L1.DIN
- removed net N$12 (its old number): L112.DIN, L113.DOUT
- removed net N$25 (its old number): L111.DIN, L112.DOUT
- removed net N$26 (its old number): L111.DOUT, L114.DIN
- removed net OUTGES: L114.DOUT
- removed net OUTROW1: L11.DOUT, L12.DIN
- removed net OUTROW10: L110.DOUT, L113.DIN
- removed net OUTROW2: L22.DOUT, L23.DIN
- removed net OUTROW3: L33.DOUT, L34.DIN
- removed net OUTROW4: L44.DOUT, L45.DIN
- removed net OUTROW5: L55.DOUT, L56.DIN
- removed net OUTROW6: L66.DOUT, L67.DIN
- removed net OUTROW7: L77.DOUT, L78.DIN
- removed net OUTROW8: L88.DOUT, L89.DIN
- removed net OUTROW9: L100.DIN, L99.DOUT
- net +5V: no longer C111.1, C112.1, C113.1, C114.1, L111.VDD, L112.VDD, L113.VDD, L114.VDD
- net GND: no longer C111.2, C112.2, C113.2, C114.2, L111.GND, L112.GND, L113.GND, L114.GND
