File: Eagle/Wordclock/Wordclock.sch (EAGLE design)
At the start: 223 parts

Commit message: Eagle Layout geroutet
Parts:
- added C111, C112, C113, C114, C115: 100n, rcl:C-EUC1310
- added C116, C117: (no value), rcl:C-EUC0805
- added IC1: MEGA8-P, atmel:MEGA8-P
- added LED1, LED2, LED3, LED4, LED5: (no value), led:LEDCHIPLED_1206
- added Q2: (no value), crystal:CRYSTALHC49S
- added R1, R2: (no value), rcl:R-EU_M0805
- added R10, R11, R12, R3, R4, R5, R6, R7, R8, R9: (no value), rcl:R-EU_M1206
- added S1, S2, S3, S4, S5: (no value), switch-omron:10-XX
- added SG1: F/HMB, buzzer:F/HMB
- added SV1: (no value), con-harting-ml:ML6L
Connections:
- removed net VCC: U$1.1
- new net INTA: R1.1, S+1.!INTA
- new net INTB: R2.1, S+1.SQW/!INTB!
- new net LEDALARM: LED5.C
- new net LEDMIN1: IC1.PB2(SS/OC1B), LED1.C
- new net LEDMIN2: IC1.PB3(MOSI/OC2), LED2.C, SV1.4
- new net LEDMIN3: IC1.PB4(MISO), LED3.C, SV1.1
- new net LEDMIN4: IC1.PB5(SCK), LED4.C, SV1.3
- new net N$103: L11.DOUT, L12.DIN
- new net N$104: L22.DOUT, L23.DIN
- new net N$105: L33.DOUT, L34.DIN
- new net N$106: L44.DOUT, L45.DIN
- new net N$107: L55.DOUT, L56.DIN
- new net N$108: L66.DOUT, L67.DIN
- new net N$109: L77.DOUT, L78.DIN
- new net N$110: L88.DOUT, L89.DIN
- new net N$111: L100.DIN, L99.DOUT
- new net N$112: C115.1, R8.1, S5.S
- new net N$113: C111.1, R9.1, S1.S
- new net N$114: LED1.A, R3.2
- new net N$115: LED2.A, R4.2
- new net N$116: LED3.A, R5.2
- new net N$117: LED4.A, R6.2
- new net N$118: LED5.A, R7.2
- new net N$119: IC1.PC4(ADC4/SDA)
- new net N$120: IC1.PC5(ADC5/SCL)
- new net N$121: IC1.PD2(INT0)
- new net N$122: IC1.PD3(INT1)
- new net N$123: C112.1, R10.1, S2.S
- new net N$124: C113.1, R11.1, S3.S
- new net N$125: C114.1, R12.1, S4.S
- new net N$126: IC1.PC0(ADC0)
- new net N$127: IC1.PC1(ADC1)
- new net N$128: IC1.PC2(ADC2)
- new net N$129: IC1.PC3(ADC3)
- new net N$130: IC1.PD0(RXD)
- new net N$131: IC1.PD1(TXD)
- new net N$132: IC1.PD4(XCK/T0)
- new net N$133: IC1.PD5(T1)
- new net N$134: IC1.PD6(AIN0)
- new net N$135: IC1.PD7(AIN1)
- new net N$136: C117.2, IC1.PB6(XTAL1/TOSC1), Q2.2
- new net N$137: C116.2, IC1.PB7(XTAL2/TOSC2), Q2.1
- new net N$141: IC1.PB1(OC1A)
- new net N$142: IC1.PB0(ICP)
- new net RESET: IC1.PC6(/RESET), SV1.5
- new net SCHALTER1: R9.2
- new net SCHALTER2: R10.2
- new net SCHALTER3: R11.2
- new net SCHALTER4: R12.2
- new net SCHALTER5: R8.2
- new net SCL: S+1.SCL
- new net SDA: S+1.SDA
- net +5V: now also IC1.AREF, IC1.AVCC, IC1.VCC@1, R1.2, R2.2, R3.1, R4.1, R5.1, R6.1, R7.1, S+1.VCC, SV1.2, U$1.1
- net GND: now also C111.2, C112.2, C113.2, C114.2, C115.2, C116.1, C117.1, IC1.GND, IC1.GND@1, S1.P, S2.P, S3.P, S4.P, S5.P, SV1.6
Other:
- note added: "Optional sechste LED für Schrift unten"
- note added: "optional zunächst"
- moved on the sheet: Q1, S+1

Commit message: Eagle VDD gelayoutet und vieles mehr
Parts:
- removed SG1: F/HMB, buzzer:F/HMB
- added C118, C119, C120: 100n, rcl:C-EUC0805
- added L111: 10u, rcl:L-EUL2012C
- added LDR, R_LED2, R_LED5: (no value), rcl:R-EU_M1206
- added PAD1, PAD2: (no value), wirepad:2,54/1,1
- added Q3: SUP75N06-08, transistor-fet:SUP75N06-08
- added SP1: AL11P, buzzer:AL11P
- Q1: device special:XTAL -> crystal:CRYSTALHC49S
- renumbered R3 to R_LED1, R5 to R_LED3, R6 to R_LED4, R7 to R_LEDAL
Connections:
- removed net N$124: C113.1, R11.1, S3.S
- removed net N$125: C114.1, R12.1, S4.S
- removed net N$128: IC1.PC2(ADC2)
- removed net N$129: IC1.PC3(ADC3)
- removed net N$130: IC1.PD0(RXD)
- removed net N$131: IC1.PD1(TXD)
- removed net N$132: IC1.PD4(XCK/T0)
- removed net N$133: IC1.PD5(T1)
- removed net N$134: IC1.PD6(AIN0)
- removed net N$135: IC1.PD7(AIN1)
- removed net N$141: IC1.PB1(OC1A)
- removed net N$142: IC1.PB0(ICP)
- new net LDR: IC1.PC3(ADC3), LDR.1, R4.2
- new net MATRIXIN: IC1.PC2(ADC2), L1.DIN
- new net MATRIXOUT: L110.DOUT
- new net NC1: IC1.PB0(ICP), PAD1.P
- new net NC2: IC1.PB1(OC1A), PAD2.P
- new net VDD: C1.1, C10.1, C100.1, C101.1, C102.1, C103.1, C104.1, C105.1, C106.1, C107.1, C108.1, C109.1, C11.1, C110.1, C12.1, C13.1, C14.1, C15.1, C16.1, C17.1, C18.1, C19.1, C2.1, C20.1, C21.1, C22.1, C23.1, C24.1, C25.1, C26.1, C27.1, C28.1, C29.1, C3.1, C30.1, C31.1, C32.1, C33.1, C34.1, C35.1, C36.1, C37.1, C38.1, C39.1, C4.1, C40.1, C41.1, C42.1, C43.1, C44.1, C45.1, C46.1, C47.1, C48.1, C49.1, C5.1, C50.1, C51.1, C52.1, C53.1, C54.1, C55.1, C56.1, C57.1, C58.1, C59.1, C6.1, C60.1, C61.1, C62.1, C63.1, C64.1, C65.1, C66.1, C67.1, C68.1, C69.1, C7.1, C70.1, C71.1, C72.1, C73.1, C74.1, C75.1, C76.1, C77.1, C78.1, C79.1, C8.1, C80.1, C81.1, C82.1, C83.1, C84.1, C85.1, C86.1, C87.1, C88.1, C89.1, C9.1, C90.1, C91.1, C92.1, C93.1, C94.1, C95.1, C96.1, C97.1, C98.1, C99.1, L1.VDD, L10.VDD, L100.VDD, L101.VDD, L102.VDD, L103.VDD, L104.VDD, L105.VDD, L106.VDD, L107.VDD, L108.VDD, L109.VDD, L11.VDD, L110.VDD, L12.VDD, L13.VDD, L14.VDD, L15.VDD, L16.VDD, L17.VDD, L18.VDD, L19.VDD, L2.VDD, L20.VDD, L21.VDD, L22.VDD, L23.VDD, L24.VDD, L25.VDD, L26.VDD, L27.VDD, L28.VDD, L29.VDD, L3.VDD, L30.VDD, L31.VDD, L32.VDD, L33.VDD, L34.VDD, L35.VDD, L36.VDD, L37.VDD, L38.VDD, L39.VDD, L4.VDD, L40.VDD, L41.VDD, L42.VDD, L43.VDD, L44.VDD, L45.VDD, L46.VDD, L47.VDD, L48.VDD, L49.VDD, L5.VDD, L50.VDD, L51.VDD, L52.VDD, L53.VDD, L54.VDD, L55.VDD, L56.VDD, L57.VDD, L58.VDD, L59.VDD, L6.VDD, L60.VDD, L61.VDD, L62.VDD, L63.VDD, L64.VDD, L65.VDD, L66.VDD, L67.VDD, L68.VDD, L69.VDD, L7.VDD, L70.VDD, L71.VDD, L72.VDD, L73.VDD, L74.VDD, L75.VDD, L76.VDD, L77.VDD, L78.VDD, L79.VDD, L8.VDD, L80.VDD, L81.VDD, L82.VDD, L83.VDD, L84.VDD, L85.VDD, L86.VDD, L87.VDD, L88.VDD, L89.VDD, L9.VDD, L90.VDD, L91.VDD, L92.VDD, L93.VDD, L94.VDD, L95.VDD, L96.VDD, L97.VDD, L98.VDD, L99.VDD, Q3.S
- net +5V: now also C120.2, L111.1, LDR.2, Q3.D, R_LED2.1, R_LED5.2, SP1.2; no longer C1.1, C10.1, C100.1, C101.1, C102.1, C103.1, C104.1, C105.1, C106.1, C107.1, C108.1, C109.1, C11.1, C110.1, C12.1, C13.1, C14.1, C15.1, C16.1, C17.1, C18.1, C19.1, C2.1, C20.1, C21.1, C22.1, C23.1, C24.1, C25.1, C26.1, C27.1, C28.1, C29.1, C3.1, C30.1, C31.1, C32.1, C33.1, C34.1, C35.1, C36.1, C37.1, C38.1, C39.1, C4.1, C40.1, C41.1, C42.1, C43.1, C44.1, C45.1, C46.1, C47.1, C48.1, C49.1, C5.1, C50.1, C51.1, C52.1, C53.1, C54.1, C55.1, C56.1, C57.1, C58.1, C59.1, C6.1, C60.1, C61.1, C62.1, C63.1, C64.1, C65.1, C66.1, C67.1, C68.1, C69.1, C7.1, C70.1, C71.1, C72.1, C73.1, C74.1, C75.1, C76.1, C77.1, C78.1, C79.1, C8.1, C80.1, C81.1, C82.1, C83.1, C84.1, C85.1, C86.1, C87.1, C88.1, C89.1, C9.1, C90.1, C91.1, C92.1, C93.1, C94.1, C95.1, C96.1, C97.1, C98.1, C99.1, IC1.AREF, IC1.AVCC, L1.VDD, L10.VDD, L100.VDD, L101.VDD, L102.VDD, L103.VDD, L104.VDD, L105.VDD, L106.VDD, L107.VDD, L108.VDD, L109.VDD, L11.VDD, L110.VDD, L12.VDD, L13.VDD, L14.VDD, L15.VDD, L16.VDD, L17.VDD, L18.VDD, L19.VDD, L2.VDD, L20.VDD, L21.VDD, L22.VDD, L23.VDD, L24.VDD, L25.VDD, L26.VDD, L27.VDD, L28.VDD, L29.VDD, L3.VDD, L30.VDD, L31.VDD, L32.VDD, L33.VDD, L34.VDD, L35.VDD, L36.VDD, L37.VDD, L38.VDD, L39.VDD, L4.VDD, L40.VDD, L41.VDD, L42.VDD, L43.VDD, L44.VDD, L45.VDD, L46.VDD, L47.VDD, L48.VDD, L49.VDD, L5.VDD, L50.VDD, L51.VDD, L52.VDD, L53.VDD, L54.VDD, L55.VDD, L56.VDD, L57.VDD, L58.VDD, L59.VDD, L6.VDD, L60.VDD, L61.VDD, L62.VDD, L63.VDD, L64.VDD, L65.VDD, L66.VDD, L67.VDD, L68.VDD, L69.VDD, L7.VDD, L70.VDD, L71.VDD, L72.VDD, L73.VDD, L74.VDD, L75.VDD, L76.VDD, L77.VDD, L78.VDD, L79.VDD, L8.VDD, L80.VDD, L81.VDD, L82.VDD, L83.VDD, L84.VDD, L85.VDD, L86.VDD, L87.VDD, L88.VDD, L89.VDD, L9.VDD, L90.VDD, L91.VDD, L92.VDD, L93.VDD, L94.VDD, L95.VDD, L96.VDD, L97.VDD, L98.VDD, L99.VDD, R4.1
- net GND: now also C118.1, C119.1, C120.1, R4.1, S1.P1, S2.P1, S3.P1, S4.P1, S5.P1
- net INTA: now also IC1.PD2(INT0)
- net INTB: now also IC1.PD3(INT1)
- net LEDALARM: now also IC1.PC0(ADC0)
- net N$112: now also IC1.PD0(RXD), SP1.1; no longer C115.1, R8.1, S5.S
- net N$113: now also C118.2, IC1.AVCC, L111.2; no longer C111.1, R9.1, S1.S
- net N$115: now also R_LED2.2; no longer R4.2
- net N$119: now also R9.1, S1.S, S1.S1; no longer IC1.PC4(ADC4/SDA)
- net N$120: now also R10.1, S2.S; no longer IC1.PC5(ADC5/SCL)
- net N$121: now also R11.1, S3.S; no longer IC1.PD2(INT0)
- net N$122: now also R12.1, S4.S; no longer IC1.PD3(INT1)
- net N$123: now also C119.2, IC1.AREF; no longer C112.1, R10.1, S2.S
- net N$126: now also R8.1, S5.S; no longer IC1.PC0(ADC0)
- net N$127: now also Q3.G
- net N$136: now also Q2.1; no longer Q2.2
- net N$137: now also Q2.2; no longer Q2.1
- net RESET: now also R_LED5.1
- net SCHALTER1: now also C111.1, IC1.PD1(TXD)
- net SCHALTER2: now also C112.1, IC1.PD4(XCK/T0)
- net SCHALTER3: now also C113.1, IC1.PD5(T1)
- net SCHALTER4: now also C114.1, IC1.PD6(AIN0)
- net SCHALTER5: now also C115.1, IC1.PD7(AIN1)
- net SCL: now also IC1.PC5(ADC5/SCL)
- net SDA: now also IC1.PC4(ADC4/SDA)
Other:
- moved on the sheet: C111, C112, C113, C114, C115, Q2, R10, R11, R12, R4, R8, R9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
